File: templog_mainboard/templog_mainboard.kicad_sch (KiCad schematic)
At the start: 3 parts, among them U1 ESP32-S3-MINI-1, U2 DS3231MZ, U3 SHT4x

Commit message: elecricity
Parts:
- added C1, C3, C4, C5: 0.1uf, Capacitor_SMD:C_0201_0603Metric, symbol Device:C
- added C2: 10uf, Capacitor_SMD:C_0201_0603Metric, symbol Device:C
- added R1, R2: 10k, symbol Device:R_US
- added U6: 24LC512, symbol Memory_EEPROM:24LC512
Connections:
- net I2C_SDA: now reaches U3.1 (SDA)
- net I2C_SDA: now also U1.31 (IO35), U2.7 (SDA), R2.1, U6.5 (SDA)
- net I2C_SCL: now reaches U3.2 (SCL)
- net I2C_SCL: now also U1.29 (IO34), U2.8 (SCL), R1.1, U6.6 (SCL)
- net +3.3V: now reaches U3.3 (VDD)
- net +3.3V: now also U1.3 (3V3), U2.6 (VBAT), C1.2, C2.2, C3.2, C4.1, C5.2, R1.2, R2.2, U6.8 (VCC)
- net GND: now reaches U3.4 (VSS)
- net GND: now also U1.1 (GND), U1.2 (GND), U1.42 (GND), U1.43 (GND), U1.46 (GND), U1.47 (GND), U1.48 (GND), U1.49 (GND), U1.50 (GND), U1.51 (GND), U1.52 (GND), U1.53 (GND), U1.54 (GND), U1.55 (GND), U1.56 (GND), U1.57 (GND), U1.58 (GND), U1.59 (GND), U1.60 (GND), U1.61 (GND), U1.62 (GND), U1.63 (GND), U1.64 (GND), U1.65 (GND), U2.2 (VCC), U2.5 (GND), C1.1, C2.1, C3.1, C4.2, C5.1, U6.1 (A0), U6.2 (A1), U6.3 (A2), U6.4 (GND), U6.7 (WP)
- no-connect marks 0 -> 3
Other:
- sheet power_mgmt ports: added +3.3Vout, CHG, ESP_SCL, ESP_SDA, USB_D-, USB_d+; removed none
- moved on the sheet: U1, U2, U3

Commit message: electtrirciy
Parts:
- added C21: 4.7uf, Capacitor_SMD:C_0201_0603Metric, symbol Device:C
- added C22: 4.7uf/50v, Capacitor_SMD:C_0201_0603Metric, symbol Device:C
- added C23: 1uf, Capacitor_SMD:C_0201_0603Metric, symbol Device:C
- added C24, C25, C26, C27, C28, C29, C30: 1uf/50v, Capacitor_SMD:C_0201_0603Metric, symbol Device:C
- added D2, D3, D4: MBR0530, Diode_SMD:D_SOD-123, symbol Diode:MBR0530
- added FPC1: FPC-05F-24PH20, FPC-05F-24PH20:FPC-SMD_24P-P0.50_FPC-05F-24PH20, symbol FPC-05F-24PH20:FPC-05F-24PH20
- added L2: 47uH, Inductor_SMD:L_6.3x6.3_H3, symbol Device:L
- added Q1: Si1308EDL, Package_TO_SOT_SMD:SOT-323_SC-70, symbol Transistor_FET:Si1308EDL
- added R16: 2.2, Resistor_SMD:R_0201_0603Metric, symbol Device:R_US
- added R17: 1M, Resistor_SMD:R_0201_0603Metric, symbol Device:R_US
- R1, R2: footprint (none) -> Resistor_SMD:R_0201_0603Metric
- U6: footprint (none) -> Package_SO:SOIC-8_3.9x4.9mm_P1.27mm
Connections:
- net +3.3V: now also C21.1, L2.1
- net GND: now also C21.2, C23.1, C24.1, C25.1, C26.1, C27.1, C28.1, C29.1, C30.1, D2.1 (K), R16.1, R17.1
- net I2C_SCL: now also FPC1.6
- net I2C_SDA: now also FPC1.7
- net dsp_busy: now reaches U1.12 (IO8)
- net dsp_busy: now also FPC1.9
- net dsp_rst: now reaches U1.13 (IO9)
- net dsp_rst: now also FPC1.10
- net dsp_dc: now reaches U1.14 (IO10)
- net dsp_dc: now also FPC1.11
- net dsp_cs: now reaches U1.15 (IO11)
- net dsp_cs: now also FPC1.12
- net dsp_sclk: now reaches U1.16 (IO12)
- net dsp_sclk: now also FPC1.13
- net dsp_sdi: now reaches U1.17 (IO13)
- net dsp_sdi: now also FPC1.14
- net USB-: now reaches U1.23 (USB_D-)
- net USB+: now reaches U1.24 (USB_D+)
- new net: C22.1, D2.2 (A), D3.1 (K)
- new net: C26.2, FPC1.20
- new net: C24.2, FPC1.15
- new net: C25.2, FPC1.18
- new net: C28.2, FPC1.22
- new net: C30.2, FPC1.24
- new net: C23.2, FPC1.5
- new net: C22.2, D4.2 (A), L2.2, Q1.3 (D)
- new net GDR: FPC1.2, Q1.1 (G), R17.2
- new net PREVGH: C27.2, D4.1 (K), FPC1.21
- new net PREVGL: C29.2, D3.2 (A), FPC1.23
- new net RESE: FPC1.3, Q1.2 (S), R16.2
- no-connect marks 3 -> 8

Commit message: time for electricity
Parts:
- L2: value 47uH -> 10uH; footprint Inductor_SMD:L_6.3x6.3_H3 -> Inductor_SMD:L_Sunlord_SWPA4030S
Changed lines of the file:
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@@
 			)
 		)
-		(property "Value" "47uH"
+		(property "Value" "10uH"
 			(at 229.87 118.11 90)
 			(effects
@@
 			)
 		)
-		(property "Footprint" "Inductor_SMD:L_6.3x6.3_H3"
+		(property "Footprint" "Inductor_SMD:L_Sunlord_SWPA4030S"
 			(at 229.87 120.65 0)
 			(effects

Commit message: electiricity
Parts:
- added SW1: K2-1109DE-D4SW-01, K2-1109DE-D4SW-01:KEY-TH_K2-1109DE-CXXW-XX, symbol K2-1109DE-D4SW-01:K2-1109DE-D4SW-01
Changed lines of the file:
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@@
+	)
+	(symbol
+		(lib_id "K2-1109DE-D4SW-01:K2-1109DE-D4SW-01")
+		(at 182.88 109.22 0)
+		(unit 1)
+		(exclude_from_sim no)
+		(in_bom yes)
+		(on_board yes)
+		(dnp no)
+		(fields_autoplaced yes)
+		(property "Reference" "SW1"
+			(at 184.15 107.9499 0)
+			(effects
+				(font
+					(size 1.27 1.27)
+				)
+				(justify left)
+			)
+		)
+		(property "Value" "K2-1109DE-D4SW-01"
+			(at 184.15 110.4899 0)
+			(effects
+				(font
+					(size 1.27 1.27)
+				)
+				(justify left)
+			)
+		)
+		(property "Footprint" "K2-1109DE-D4SW-01:KEY-TH_K2-1109DE-CXXW-XX"
+			(at 182.88 127 0)
+			(effects
+				(font
+					(size 1.27 1.27)
+				)
+				(hide yes)
+			)
+		)
+		(property "Datasheet" "https://lcsc.com/product-detail/Tactile-Switches_Korean-Hroparts-Elec-K2-1109DE-D4SW-01_C223806.html"
+			(at 182.88 129.54 0)
+			(effects
+				(font
+					(size 1.27 1.27)
+				)
+				(hide yes)
+			)
+		)
+		(property "Description" ""
+			(at 182.88 109.22 0)
+			(effects
+				(font
+					(size 1.27 1.27)
+				)
+				(hide yes)
+			)
+		)
+		(property "LCSC Part" "C223806"
+			(at 182.88 132.08 0)
+			(effects
+				(font
+					(size 1.27 1.27)
+				)
+				(hide yes)
+			)
+		)
+		(pin "1"
+		)
+		(pin "3"
+		)
+		(pin "2"
+		)
+		(instances
+			(project ""
+				(path "/84b25dc3-cc11-42e1-888d-24c6d5a62713"
+					(reference "SW1")
+					(unit 1)
+				)
+			)
+		)
 	)
 	(symbol

Commit message: Taseotlkauset
Parts:
- removed FPC1: FPC-05F-24PH20, FPC-05F-24PH20:FPC-SMD_24P-P0.50_FPC-05F-24PH20, symbol FPC-05F-24PH20:FPC-05F-24PH20
- added C13: 1uf, Capacitor_SMD:C_0201_0603Metric, symbol Device:C
- added C14: 0.1uf, Capacitor_SMD:C_0201_0603Metric, symbol Device:C
- added FPC1: AFC07-S24ECA-00, FPC-SMD_AFC07-S24ECA-00:FPC-SMD_AFC07-S24ECA-00, symbol FPC-SMD_AFC07-S24ECA-00:AFC07-S24ECA-00
- added SW2: K2-1109DE-D4SW-01, K2-1109DE-D4SW-01:KEY-TH_K2-1109DE-CXXW-XX, symbol K2-1109DE-D4SW-01:K2-1109DE-D4SW-01
- added U9: LTC2954CTS8-2_TRMPBF, LTC2954CTS8_2_TRMPBF:TSOT-23_TS8, symbol LTC2954CTS8_2_TRMPBF:LTC2954CTS8-2_TRMPBF
Connections:
- net GDR: now also FPC1.2
- net GND: now also SW1.2, SW1.3, C13.2, C14.2, SW2.2, SW2.3, U9.4 (GND)
- net I2C_SCL: now also FPC1.6
- net I2C_SDA: now also FPC1.7
- net PREVGH: now also FPC1.21
- net PREVGL: now also FPC1.23
- net RESE: now also FPC1.3
- net dsp_busy: now also FPC1.9
- net dsp_cs: now also FPC1.12
- net dsp_dc: now also FPC1.11
- net dsp_rst: now also FPC1.10
- net dsp_sclk: now also FPC1.13
- net dsp_sdi: now also FPC1.14
- net at C26.2: now also FPC1.20
- net at C24.2: now also FPC1.15
- net at C25.2: now also FPC1.18
- net at C28.2: now also FPC1.22
- net at C30.2: now also FPC1.24
- net at C23.2: now also FPC1.5
- net power_btn: now reaches SW1.1
- net power_btn: now also U9.2 (*PB)
- new net: C13.1, U9.7 (PDT)
- new net VBattery: C14.1, U9.1 (VIN)
- new net btn_int: U9.5 (*INT)
- new net power_kill: U9.8 (*KILL)
- new net powerpath_enable: U9.6 (EN/*EN)
- no-connect marks 8 -> 9
Other:
- sheet power_mgmt ports: added +battery, SYSOFF; removed none
- moved on the sheet: R1, R2

Commit message: okay
Parts:
- added C15: 1uf, Capacitor_SMD:C_0201_0603Metric, symbol Device:C
- added R18: 10k, Resistor_SMD:R_0201_0603Metric, symbol Device:R_US
- added TP1: +RESET, TestPoint:TestPoint_Pad_1.0x1.0mm, symbol Connector:TestPoint
- added TP2: -RESET, TestPoint:TestPoint_Pad_1.0x1.0mm, symbol Connector:TestPoint
- added TP3: BOOT, TestPoint:TestPoint_Pad_1.0x1.0mm, symbol Connector:TestPoint
Connections:
- net +3.3V: now also R18.1
- net GND: now also SW1.1, C15.2, TP2.1; no longer SW1.2
- net dsp_cs: now also U1.9 (IO5); no longer U1.15 (IO11)
- net dsp_dc: now also U1.10 (IO6); no longer U1.14 (IO10)
- net dsp_rst: now also U1.11 (IO7); no longer U1.13 (IO9)
- net dsp_sclk: now also U1.8 (IO4); no longer U1.16 (IO12)
- net dsp_sdi: now also U1.7 (IO3); no longer U1.17 (IO13)
- net power_btn: now also SW1.2; no longer SW1.1
- net power_kill: now also U1.36 (IO40)
- net menu_btn: now reaches SW2.1
- net menu_btn: now also U1.6 (IO2)
- net at U1.4 (IO0): now also TP3.1
- net at U1.45 (EN): now also C15.1, R18.2, TP1.1
- no-connect marks 9 -> 11
Other:
- moved on the sheet: C23, C24, C25, C26, C27, C28, C29, C30, FPC1, SW1, SW2

Commit message: idk
Parts:
- added RST1: +RESET, TestPoint:TestPoint_Pad_2.0x2.0mm, symbol Connector:TestPoint
Connections:
- net at C15.1, R18.2, TP1.1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: now also RST1.1
Other:
- moved on the sheet: C13, C14, C3, C4, C5, R1, R2, SW1, SW2, U2, U3, U6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

Commit message: asejkthas
Parts:
- C1, C13, C15, C2, C21, C22, C23, C24, C25, C26, C27, C28, C29, C3, C30, C4, C5: footprint Capacitor_SMD:C_0201_0603Metric -> Capacitor_SMD:C_0402_1005Metric
- R1, R16, R17, R2: footprint Resistor_SMD:R_0201_0603Metric -> Resistor_SMD:R_0402_1005Metric
Changed lines of the file:
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@@
 			)
 		)
-		(property "Footprint" "Capacitor_SMD:C_0201_0603Metric"
+		(property "Footprint" "Capacitor_SMD:C_0402_1005Metric"
 			(at 140.97 105.7148 0)
 			(effects
@@
 			)
 		)
-		(property "Footprint" "Capacitor_SMD:C_0201_0603Metric"
+		(property "Footprint" "Capacitor_SMD:C_0402_1005Metric"
 			(at 218.44 67.6148 0)
 			(effects
@@
 			)
 		)
-		(property "Footprint" "Capacitor_SMD:C_0201_0603Metric"
+		(property "Footprint" "Capacitor_SMD:C_0402_1005Metric"
 			(at 160.02 29.5148 0)
 			(effects
@@
 			)
 		)
-		(property "Footprint" "Resistor_SMD:R_0201_0603Metric"
+		(property "Footprint" "Resistor_SMD:R_0402_1005Metric"
 			(at 231.394 148.336 90)
 			(effects
@@
 			)
 		)
-		(property "Footprint" "Resistor_SMD:R_0201_0603Metric"
+		(property "Footprint" "Resistor_SMD:R_0402_1005Metric"
 			(at 241.554 148.336 90)
 			(effects
@@
 			)
 		)
-		(property "Footprint" "Capacitor_SMD:C_0201_0603Metric"
+		(property "Footprint" "Capacitor_SMD:C_0402_1005Metric"
 			(at 218.44 29.5148 0)
 			(effects
@@
 			)
 		)
-		(property "Footprint" "Capacitor_SMD:C_0201_0603Metric"
+		(property "Footprint" "Capacitor_SMD:C_0402_1005Metric"
 			(at 137.16 176.8348 0)
 			(effects
@@
 			)
 		)
-		(property "Footprint" "Resistor_SMD:R_0201_0603Metric"
+		(property "Footprint" "Resistor_SMD:R_0402_1005Metric"
 			(at 103.124 122.174 90)
 			(effects
@@
 			)
 		)
-		(property "Footprint" "Capacitor_SMD:C_0201_0603Metric"
+		(property "Footprint" "Capacitor_SMD:C_0402_1005Metric"
 			(at 220.6752 132.08 0)
 			(effects
@@
 			)
 		)
-		(property "Footprint" "Capacitor_SMD:C_0201_0603Metric"
+		(property "Footprint" "Capacitor_SMD:C_0402_1005Metric"
 			(at 142.24 71.4248 0)
 			(effects
@@
 			)
 		)
-		(property "Footprint" "Capacitor_SMD:C_0201_0603Metric"
+		(property "Footprint" "Capacitor_SMD:C_0402_1005Metric"
 			(at 243.5352 113.03 0)
 			(effects
@@
 			)
 		)
-		(property "Footprint" "Capacitor_SMD:C_0201_0603Metric"
+		(property "Footprint" "Capacitor_SMD:C_0402_1005Metric"
 			(at 218.44 70.1548 0)
 			(effects
@@
 			)
 		)
-		(property "Footprint" "Capacitor_SMD:C_0201_0603Metric"
+		(property "Footprint" "Capacitor_SMD:C_0402_1005Metric"
 			(at 218.44 72.6948 0)
 			(effects
@@
 			)
 		)
-		(property "Footprint" "Capacitor_SMD:C_0201_0603Metric"
+		(property "Footprint" "Capacitor_SMD:C_0402_1005Metric"
 			(at 59.69 39.6748 0)
 			(effects
@@
 			)
 		)
-		(property "Footprint" "Capacitor_SMD:C_0201_0603Metric"
+		(property "Footprint" "Capacitor_SMD:C_0402_1005Metric"
 			(at 218.44 75.2348 0)
 			(effects
@@
 			)
 		)
-		(property "Footprint" "Capacitor_SMD:C_0201_0603Metric"
+		(property "Footprint" "Capacitor_SMD:C_0402_1005Metric"
 			(at 30.1752 59.69 0)
 			(effects
@@
 			)
 		)
-		(property "Footprint" "Capacitor_SMD:C_0201_0603Metric"
+		(property "Footprint" "Capacitor_SMD:C_0402_1005Metric"
 			(at 218.44 54.9148 0)
 			(effects
@@
 			)
 		)
-		(property "Footprint" "Resistor_SMD:R_0201_0603Metric"
+		(property "Footprint" "Resistor_SMD:R_0402_1005Metric"
 			(at 103.124 110.744 90)
 			(effects
@@
 			)
 		)
-		(property "Footprint" "Capacitor_SMD:C_0201_0603Metric"
+		(property "Footprint" "Capacitor_SMD:C_0402_1005Metric"
 			(at 59.69 28.2448 0)
 			(effects
@@
 			)
 		)
-		(property "Footprint" "Capacitor_SMD:C_0201_0603Metric"
+		(property "Footprint" "Capacitor_SMD:C_0402_1005Metric"
 			(at 218.44 62.5348 0)
 			(effects
@@
 			)
 		)
-		(property "Footprint" "Capacitor_SMD:C_0201_0603Metric"
+		(property "Footprint" "Capacitor_SMD:C_0402_1005Metric"
 			(at 218.44 77.7748 0)
 			(effects
