File: templog_mainboard/templog_mainboard.kicad_sch (KiCad schematic)
At the start: 40 parts, among them Q1 Si1308EDL, SW1 K2-1109DE-D4SW-01, SW2 K2-1109DE-D4SW-01, U1 ESP32-S3-MINI-1, U2 DS3231MZ, U3 SHT4x, U6 24LC512, U9 LTC2954CTS8-2_TRMPBF

Commit message: laout
Parts:
- removed RST1: +RESET, TestPoint:TestPoint_Pad_2.0x2.0mm, symbol Connector:TestPoint
- C14: footprint Capacitor_SMD:C_0201_0603Metric -> Capacitor_SMD:C_0402_1005Metric
- R18: footprint Resistor_SMD:R_0201_0603Metric -> Resistor_SMD:R_0402_1005Metric
Changed lines of the file:
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@@
 	)
 	(junction
-		(at 25.4 50.8)
-		(diameter 0)
-		(color 0 0 0 0)
-	)
-	(junction
 		(at 29.21 50.8)
 		(diameter 0)
@@
 	(wire
 		(pts
-			(xy 25.4 50.8) (xy 29.21 50.8)
+			(xy 21.59 50.8) (xy 29.21 50.8)
 		)
 		(stroke
@@
 	(wire
 		(pts
-			(xy 21.59 41.91) (xy 25.4 41.91)
-		)
-		(stroke
-			(width 0)
-			(type default)
-		)
-	)
-	(wire
-		(pts
 			(xy 133.35 106.68) (xy 132.08 106.68)
 		)
@@
 	(wire
 		(pts
-			(xy 21.59 50.8) (xy 25.4 50.8)
-		)
-		(stroke
-			(width 0)
-			(type default)
-		)
-	)
-	(wire
-		(pts
 			(xy 120.65 181.61) (xy 120.65 177.8)
 		)
@@
 	(wire
 		(pts
-			(xy 25.4 41.91) (xy 25.4 50.8)
-		)
-		(stroke
-			(width 0)
-			(type default)
-		)
-	)
-	(wire
-		(pts
 			(xy 218.44 68.58) (xy 241.3 68.58)
 		)
@@
 			)
 		)
-		(property "Footprint" "Capacitor_SMD:C_0201_0603Metric"
+		(property "Footprint" "Capacitor_SMD:C_0402_1005Metric"
 			(at 53.6448 170.18 0)
 			(effects
@@
 			)
 		)
-		(property "Footprint" "Resistor_SMD:R_0201_0603Metric"
+		(property "Footprint" "Resistor_SMD:R_0402_1005Metric"
 			(at 30.226 43.434 90)
 			(effects
@@
 					(unit 1)
 				)
-			)
-		)
-	)
-	(symbol
-		(lib_id "Connector:TestPoint")
-		(at 21.59 41.91 90)
-		(unit 1)
-		(exclude_from_sim no)
-		(in_bom yes)
-		(on_board yes)
-		(dnp no)
-		(fields_autoplaced yes)
-		(property "Reference" "RST1"
-			(at 18.288 36.83 90)
-			(effects
-				(font
-					(size 1.27 1.27)
-				)
-			)
-		)
-		(property "Value" "+RESET"
-			(at 18.288 39.37 90)
-			(effects
-				(font
-					(size 1.27 1.27)
-				)
-			)
-		)
-		(property "Footprint" "TestPoint:TestPoint_Pad_2.0x2.0mm"
-			(at 21.59 36.83 0)
-			(effects
-				(font
-					(size 1.27 1.27)
-				)
-				(hide yes)
-			)
-		)
-		(property "Datasheet" "~"
-			(at 21.59 36.83 0)
-			(effects
-				(font
-					(size 1.27 1.27)
-				)
-				(hide yes)
-			)
-		)
-		(property "Description" "test point"
-			(at 21.59 41.91 0)
-			(effects
-				(font
-					(size 1.27 1.27)
-				)
-				(hide yes)
-			)
-		)
-		(pin "1"
-		)
-		(instances
-			(project "templog_mainboard"
-				(path "/84b25dc3-cc11-42e1-888d-24c6d5a62713"
-					(reference "RST1")
-					(unit 1)
-				)

Commit message: this is an electricity PCB
Connections:
- net +3.3V: now also FPC1.16
- net GND: now also FPC1.17, FPC1.8
- net I2C_SCL: no longer FPC1.6
- net I2C_SDA: no longer FPC1.7
- net btn_int: now also U1.32 (IO36)
- net power_kill: now also U1.33 (IO37); no longer U1.36 (IO40)
- net clock_alarm: now reaches U2.3 (~{INT}/SQW)
- net clock_alarm: now also U1.13 (IO9)
- net charging_status: now reaches U1.28 (IO33)
- no-connect marks 11 -> 12
Other:
- note added: "E-Ink display"
- note added: "Real time clock"
- note added: "Soft power switch latch"
- note added: "Temperature sensor"
- moved on the sheet: C3, C4, R1, R2, SW1, SW2, U2, U3

Commit message: electroscity
Parts:
- added R9: 10k, Resistor_SMD:R_0402_1005Metric, symbol Device:R_US
- C2: footprint Capacitor_SMD:C_0402_1005Metric -> Capacitor_SMD:C_0603_1608Metric
Connections:
- net +3.3V: now also R9.1
- net clock_alarm: now also U1.25 (IO21), R9.2; no longer U1.13 (IO9)
Changed lines of the file:
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@@
 	)
 	(junction
+		(at 181.61 58.42)
+		(diameter 0)
+		(color 0 0 0 0)
+	)
+	(junction
 		(at 132.08 120.65)
 		(diameter 0)
@@
 	(wire
 		(pts
+			(xy 181.61 46.99) (xy 181.61 58.42)
+		)
+		(stroke
+			(width 0)
+			(type default)
+		)
+	)
+	(wire
+		(pts
 			(xy 162.56 36.83) (xy 162.56 45.72)
 		)
@@
 	(wire
 		(pts
+			(xy 181.61 33.02) (xy 181.61 39.37)
+		)
+		(stroke
+			(width 0)
+			(type default)
+		)
+	)
+	(wire
+		(pts
 			(xy 133.35 115.57) (xy 132.08 115.57)
 		)
@@
 	(wire
 		(pts
+			(xy 81.28 63.5) (xy 85.09 63.5)
+		)
+		(stroke
+			(width 0)
+			(type default)
+		)
+	)
+	(wire
+		(pts
 			(xy 133.35 106.68) (xy 132.08 106.68)
 		)
@@
 	(wire
 		(pts
+			(xy 181.61 58.42) (xy 185.42 58.42)
+		)
+		(stroke
+			(width 0)
+			(type default)
+		)
+	)
+	(wire
+		(pts
 			(xy 236.22 50.8) (xy 241.3 50.8)
 		)
@@
 	(wire
 		(pts
-			(xy 46.99 78.74) (xy 50.8 78.74)
-		)
-		(stroke
-			(width 0)
-			(type default)
-		)
-	)
-	(wire
-		(pts
 			(xy 107.95 128.27) (xy 113.03 128.27)
 		)
@@
 	)
 	(label "clock_alarm"
-		(at 181.61 58.42 0)
+		(at 185.42 58.42 0)
 		(effects
 			(font
@@
 	)
 	(label "clock_alarm"
-		(at 46.99 78.74 180)
+		(at 85.09 63.5 0)
 		(effects
 			(font
 				(size 1.27 1.27)
 			)
-			(justify right bottom)
+			(justify left bottom)
 		)
 	)
@@
 	)
 	(symbol
+		(lib_id "power:+3.3V")
+		(at 181.61 33.02 0)
+		(unit 1)
+		(exclude_from_sim no)
+		(in_bom yes)
+		(on_board yes)
+		(dnp no)
+		(fields_autoplaced yes)
+		(property "Reference" "#PWR054"
+			(at 181.61 36.83 0)
+			(effects
+				(font
+					(size 1.27 1.27)
+				)
+				(hide yes)
+			)
+		)
+		(property "Value" "+3.3V"
+			(at 181.61 27.94 0)
+			(effects
+				(font
+					(size 1.27 1.27)
+				)
+			)
+		)
+		(property "Footprint" ""
+			(at 181.61 33.02 0)
+			(effects
+				(font
+					(size 1.27 1.27)
+				)
+				(hide yes)
+			)
+		)
+		(property "Datasheet" ""
+			(at 181.61 33.02 0)
+			(effects
+				(font
+					(size 1.27 1.27)
+				)
+				(hide yes)
+			)
+		)
+		(property "Description" "Power symbol creates a global label with name \"+3.3V\""
+			(at 181.61 33.02 0)
+			(effects
+				(font
+					(size 1.27 1.27)
+				)
+				(hide yes)
+			)
+		)
+		(pin "1"
+		)
+		(instances
+			(project "templog_mainboard"
+				(path "/84b25dc3-cc11-42e1-888d-24c6d5a62713"
+					(reference "#PWR054")
+					(unit 1)
+				)
+			)
+		)
+	)
+	(symbol
 		(lib_id "Device:C")
 		(at 158.75 36.83 90)
@@
 			)
 		)
-		(property "Footprint" "Capacitor_SMD:C_0402_1005Metric"
+		(property "Footprint" "Capacitor_SMD:C_0603_1608Metric"
 			(at 59.69 39.6748 0)
 			(effects
@@
 					(unit 1)
 				)
+			)
+		)
+	)
+	(symbol
+		(lib_id "Device:R_US")
+		(at 181.61 43.18 0)
+		(unit 1)
+		(exclude_from_sim no)
+		(in_bom yes)
+		(on_board yes)
+		(dnp no)
+		(fields_autoplaced yes)
+		(property "Reference" "R9"
+			(at 184.15 41.9099 0)
+			(effects
+				(font
+					(size 1.27 1.27)
+				)
+				(justify left)
+			)
+		)
+		(property "Value" "10k"
+			(at 184.15 44.4499 0)
+			(effects
+				(font
+					(size 1.27 1.27)
+				)
+				(justify left)
+			)
+		)
+		(property "Footprint" "Resistor_SMD:R_0402_1005Metric"
+			(at 182.626 43.434 90)
+			(effects
+				(font
+					(size 1.27 1.27)
+				)
+				(hide yes)
+			)
+		)
+		(property "Datasheet" "~"
+			(at 181.61 43.18 0)
+			(effects
+				(font
+					(size 1.27 1.27)
+				)
+				(hide yes)
+			)
+		)
+		(property "Description" "Resistor, US symbol"
+			(at 181.61 43.18 0)
+			(effects
+				(font
+					(size 1.27 1.27)
+				)
+				(hide yes)
+			)
+		)
+		(pin "1"
+		)
+		(pin "2"
+		)
+		(instances
+			(project "templog_mainboard"
+				(path "/84b25dc3-cc11-42e1-888d-24c6d5a62713"
+					(reference "R9")
+					(unit 1)
+				)

Commit message: :ASEDfasef
Parts:
- C2: footprint Capacitor_SMD:C_0603_1608Metric -> Capacitor_SMD:C_0805_2012Metric
- C21, C22: footprint Capacitor_SMD:C_0402_1005Metric -> Capacitor_SMD:C_0603_1608Metric
Changed lines of the file:
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@@
 			)
 		)
-		(property "Footprint" "Capacitor_SMD:C_0402_1005Metric"
+		(property "Footprint" "Capacitor_SMD:C_0603_1608Metric"
 			(at 220.6752 132.08 0)
 			(effects
@@
 			)
 		)
-		(property "Footprint" "Capacitor_SMD:C_0402_1005Metric"
+		(property "Footprint" "Capacitor_SMD:C_0603_1608Metric"
 			(at 243.5352 113.03 0)
 			(effects
@@
 			)
 		)
-		(property "Footprint" "Capacitor_SMD:C_0603_1608Metric"
+		(property "Footprint" "Capacitor_SMD:C_0805_2012Metric"
 			(at 59.69 39.6748 0)
 			(effects

Commit message: electractiyt
Parts:
- C13, C23, C24, C25, C26, C27, C28, C29, C30: footprint Capacitor_SMD:C_0402_1005Metric -> Capacitor_SMD:C_0603_1608Metric
Connections:
- net dsp_busy: now also U1.15 (IO11); no longer U1.12 (IO8)
- net dsp_cs: now also U1.12 (IO8); no longer U1.9 (IO5)
- net dsp_dc: now also U1.13 (IO9); no longer U1.10 (IO6)
- net dsp_rst: now also U1.14 (IO10); no longer U1.11 (IO7)
- net dsp_sclk: now also U1.11 (IO7); no longer U1.8 (IO4)
- net dsp_sdi: now also U1.10 (IO6); no longer U1.7 (IO3)
Changed lines of the file:
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@@
 	(wire
 		(pts
-			(xy 133.35 106.68) (xy 132.08 106.68)
+			(xy 46.99 71.12) (xy 50.8 71.12)
 		)
 		(stroke
@@
 	(wire
 		(pts
-			(xy 181.61 58.42) (xy 185.42 58.42)
+			(xy 133.35 106.68) (xy 132.08 106.68)
 		)
 		(stroke
@@
 	(wire
 		(pts
-			(xy 236.22 50.8) (xy 241.3 50.8)
+			(xy 181.61 58.42) (xy 185.42 58.42)
 		)
 		(stroke
@@
 	(wire
 		(pts
-			(xy 54.61 166.37) (xy 54.61 170.18)
+			(xy 236.22 50.8) (xy 241.3 50.8)
 		)
 		(stroke
@@
 	(wire
 		(pts
-			(xy 59.69 124.46) (xy 66.04 124.46)
+			(xy 54.61 166.37) (xy 54.61 170.18)
 		)
 		(stroke
@@
 	(wire
 		(pts
-			(xy 236.22 22.86) (xy 241.3 22.86)
+			(xy 59.69 124.46) (xy 66.04 124.46)
 		)
 		(stroke
@@
 	(wire
 		(pts
-			(xy 218.44 76.2) (xy 241.3 76.2)
+			(xy 236.22 22.86) (xy 241.3 22.86)
 		)
 		(stroke
@@
 	(wire
 		(pts
-			(xy 132.08 118.11) (xy 133.35 118.11)
+			(xy 218.44 76.2) (xy 241.3 76.2)
 		)
 		(stroke
@@
 	(wire
 		(pts
-			(xy 46.99 76.2) (xy 50.8 76.2)
+			(xy 132.08 118.11) (xy 133.35 118.11)
 		)
 		(stroke
@@
 	(wire
 		(pts
-			(xy 46.99 73.66) (xy 50.8 73.66)
-		)
-		(stroke
-			(width 0)
-			(type default)
-		)
-	)
-	(wire
-		(pts
 			(xy 201.93 68.58) (xy 210.82 68.58)
 		)
@@
 	(wire
 		(pts
+			(xy 46.99 78.74) (xy 50.8 78.74)
+		)
+		(stroke
+			(width 0)
+			(type default)
+		)
+	)
+	(wire
+		(pts
 			(xy 201.93 71.12) (xy 210.82 71.12)
 		)
@@
 	(wire
 		(pts
+			(xy 46.99 73.66) (xy 50.8 73.66)
+		)
+		(stroke
+			(width 0)
+			(type default)
+		)
+	)
+	(wire
+		(pts
 			(xy 232.41 129.54) (xy 234.95 129.54)
 		)
@@
 	(wire
 		(pts
-			(xy 46.99 68.58) (xy 50.8 68.58)
+			(xy 59.69 29.21) (xy 66.04 29.21)
 		)
 		(stroke
@@
 	(wire
 		(pts
-			(xy 59.69 29.21) (xy 66.04 29.21)
+			(xy 242.57 140.97) (xy 242.57 144.78)
 		)
 		(stroke
@@
 	(wire
 		(pts
-			(xy 242.57 140.97) (xy 242.57 144.78)
+			(xy 218.44 55.88) (xy 241.3 55.88)
 		)
 		(stroke
@@
 	(wire
 		(pts
-			(xy 218.44 55.88) (xy 241.3 55.88)
+			(xy 46.99 76.2) (xy 50.8 76.2)
 		)
 		(stroke
@@
 	(wire
 		(pts
-			(xy 46.99 63.5) (xy 50.8 63.5)
+			(xy 81.28 71.12) (xy 85.09 71.12)
 		)
 		(stroke
@@
 	(wire
 		(pts
-			(xy 81.28 71.12) (xy 85.09 71.12)
+			(xy 46.99 81.28) (xy 50.8 81.28)
 		)
 		(stroke
@@
 	(wire
 		(pts
-			(xy 46.99 71.12) (xy 50.8 71.12)
-		)
-		(stroke
-			(width 0)
-			(type default)
-		)
-	)
-	(wire
-		(pts
 			(xy 218.44 73.66) (xy 241.3 73.66)
 		)
@@
 	(wire
 		(pts
-			(xy 46.99 66.04) (xy 50.8 66.04)
-		)
-		(stroke
-			(width 0)
-			(type default)
-		)
-	)
-	(wire
-		(pts
 			(xy 123.19 73.66) (xy 123.19 76.2)
 		)
@@
 	(wire
 		(pts
+			(xy 46.99 83.82) (xy 50.8 83.82)
+		)
+		(stroke
+			(width 0)
+			(type default)
+		)
+	)
+	(wire
+		(pts
 			(xy 29.21 36.83) (xy 29.21 39.37)
 		)
@@
 	)
 	(label "dsp_dc"
-		(at 46.99 71.12 180)
+		(at 46.99 78.74 180)
 		(effects
 			(font
@@
 	)
 	(label "dsp_busy"
-		(at 46.99 76.2 180)
+		(at 46.99 83.82 180)
 		(effects
 			(font
@@
 	)
 	(label "dsp_sclk"
-		(at 46.99 66.04 180)
+		(at 46.99 73.66 180)
 		(effects
 			(font
@@
 	)
 	(label "dsp_sdi"
-		(at 46.99 63.5 180)
+		(at 46.99 71.12 180)
 		(effects
 			(font
@@
 	)
 	(label "dsp_rst"
-		(at 46.99 73.66 180)
+		(at 46.99 81.28 180)
 		(effects
 			(font
@@
 	)
 	(label "dsp_cs"
-		(at 46.99 68.58 180)
+		(at 46.99 76.2 180)
 		(effects
 			(font
@@
 			)
 		)
-		(property "Footprint" "Capacitor_SMD:C_0402_1005Metric"
+		(property "Footprint" "Capacitor_SMD:C_0603_1608Metric"
 			(at 218.44 67.6148 0)
 			(effects
@@
 			)
 		)
-		(property "Footprint" "Capacitor_SMD:C_0402_1005Metric"
+		(property "Footprint" "Capacitor_SMD:C_0603_1608Metric"
 			(at 218.44 29.5148 0)
 			(effects
@@
 			)
 		)
-		(property "Footprint" "Capacitor_SMD:C_0402_1005Metric"
+		(property "Footprint" "Capacitor_SMD:C_0603_1608Metric"
 			(at 137.16 176.8348 0)
 			(effects
@@
 			)
 		)
-		(property "Footprint" "Capacitor_SMD:C_0402_1005Metric"
+		(property "Footprint" "Capacitor_SMD:C_0603_1608Metric"
 			(at 218.44 70.1548 0)
 			(effects
@@
 			)
 		)
-		(property "Footprint" "Capacitor_SMD:C_0402_1005Metric"
+		(property "Footprint" "Capacitor_SMD:C_0603_1608Metric"
 			(at 218.44 72.6948 0)
 			(effects
@@
 			)
 		)
-		(property "Footprint" "Capacitor_SMD:C_0402_1005Metric"
+		(property "Footprint" "Capacitor_SMD:C_0603_1608Metric"
 			(at 218.44 75.2348 0)
 			(effects
@@
 			)
 		)
-		(property "Footprint" "Capacitor_SMD:C_0402_1005Metric"
+		(property "Footprint" "Capacitor_SMD:C_0603_1608Metric"
 			(at 218.44 54.9148 0)
 			(effects
@@
 			)
 		)
-		(property "Footprint" "Capacitor_SMD:C_0402_1005Metric"
+		(property "Footprint" "Capacitor_SMD:C_0603_1608Metric"
 			(at 218.44 62.5348 0)
 			(effects
@@
 			)
 		)
-		(property "Footprint" "Capacitor_SMD:C_0402_1005Metric"
+		(property "Footprint" "Capacitor_SMD:C_0603_1608Metric"
 			(at 218.44 77.7748 0)
 			(effects
