File: templog_mainboard/templog_mainboard.kicad_pcb (KiCad board)
At the start: 4 copper layers, 57 parts, among them J1 USB_C_Receptacle_USB2.0_16P, J3 battery_con, Q1 Si1308EDL, U1 ESP32-S3-MINI-1, U2 DS3231MZ, U3 SHT4x, U4 BQ27441-G1, U5 BQ24075RGT, U6 24LC512, U7 USBLC6-2SC6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

Commit message: time for electricity
Parts:
- removed D1: D, Diode_SMD:D_0201_0603Metric
- added SSB43L1: D, Diode_SMD:D_SMB, F.Cu at (160.6, 57.2)
- L1: footprint Inductor_SMD:L_6.3x6.3_H3 -> Inductor_SMD:L_Sunlord_SWPA4030S
- L2: value 47uH -> 10uH; footprint Inductor_SMD:L_6.3x6.3_H3 -> Inductor_SMD:L_Sunlord_SWPA4030S
- moved U3 104.8 mm to (166.8, 50.8), turned to 90 degrees
- moved C4 104.8 mm to (166.8, 49.0), turned to 180 degrees
- moved L1 93.2 mm to (159.4, 43.0), turned to 90 degrees
- moved FPC1 76.2 mm to (132.2, 48.6), turned to -90 degrees
- moved R2 71.9 mm to (159.2, 59.8), turned to 180 degrees
- moved R1 69.8 mm to (159.2, 61.0), turned to 180 degrees
- moved C23 69.0 mm to (135.6, 45.4)
- moved C3 66.9 mm to (159.9, 66.6)
- moved C24 66.8 mm to (135.5, 49.8)
- moved U2 66.4 mm to (164.1, 68.0)
- moved C25 66.2 mm to (135.5, 50.6)
- moved C26 65.8 mm to (135.5, 51.4)
- moved C11 65.5 mm to (162.4, 42.3), turned to 90 degrees
- moved C27 65.4 mm to (135.5, 52.2)
- moved C28 65.1 mm to (135.5, 53.0)
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Connections:
- C11 pad 2: unconnected-(C11-Pad2) -> GND
- C12 pad 2: unconnected-(C12-Pad2) -> GND
Routing:
- net GND: track 10.2 -> 66.3 mm, vias 3 -> 36
- net /I2C_SCL: track 0.00 -> 22.4 mm, vias 0 -> 1
- net /power_mgmt/powerpath_out: track 0.00 -> 21.2 mm, vias 0 -> 2
- net /power_mgmt/battery_in: track 0.00 -> 21.2 mm, vias 0 -> 1
- net /I2C_SDA: track 0.00 -> 20.7 mm, vias 0 -> 2
- net +3.3V: track 0.00 -> 17.1 mm, vias 0 -> 4
- net Net-(SSB43L1-K): track 0.00 -> 14.7 mm
- net /USB-: track 15.6 -> 20.9 mm
- net /RESE: track 0.00 -> 4.79 mm
- net /USB+: track 14.2 -> 18.9 mm
- net /GDR: track 0.00 -> 4.56 mm
- net Net-(U8-FB): track 0.00 -> 4.11 mm
- net Net-(U8-BST): track 0.00 -> 2.78 mm
- net Net-(C26-Pad2): track 0.00 -> 2.33 mm
- net Net-(C25-Pad2): track 0.00 -> 2.24 mm
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
Commit message: electiricity
Parts:
- added SW1: K2-1109DE-D4SW-01, K2-1109DE-D4SW-01:KEY-TH_K2-1109DE-CXXW-XX, F.Cu at (161.1, 41.7)
- moved C22 18.3 mm to (135.4, 63.8), turned to 180 degrees
- moved C21 16.9 mm to (133.2, 63.8), turned to 0 degrees
- moved L1 14.6 mm to (160.8, 57.5), turned to -90 degrees
- moved C12 12.2 mm to (160.8, 54.2), turned to 0 degrees
- moved R12 11.1 mm to (159.2, 54.2), turned to 0 degrees
- moved C11 11.0 mm to (160.8, 53.2), turned to 0 degrees
- moved R11 9.83 mm to (159.2, 53.2), turned to 180 degrees
- moved U3 9.07 mm to (166.2, 41.8), turned to -90 degrees
- moved D2 8.24 mm to (141.0, 56.8), turned to -90 degrees
- moved C9 7.67 mm to (166.8, 50.0), turned to -90 degrees
- moved R13 7.53 mm to (166.8, 48.4), turned to 90 degrees
- moved C10 6.17 mm to (162.5, 53.2), turned to -90 degrees
- moved C4 5.69 mm to (166.3, 43.4), turned to 0 degrees
- moved Q1 4.75 mm to (137.8, 48.5), turned to -90 degrees
- moved SSB43L1 4.75 mm to (165.2, 56.2), turned to 90 degrees
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Routing:
- net /I2C_SCL: track 22.4 -> 90.7 mm, vias 1 -> 5
- net /I2C_SDA: track 20.7 -> 82.7 mm, vias 2 -> 6
- net GND: track 66.3 -> 116.3 mm, vias 36 -> 48
- net Net-(D4-A): track 0.00 -> 20.1 mm
- net /power_mgmt/V_battery: track 1.27 -> 15.6 mm, vias 0 -> 2
- net Net-(D2-A): track 0.00 -> 10.5 mm
- net /PREVGH: track 1.96 -> 11.4 mm
- net +3.3V: track 17.1 -> 24.1 mm, vias 4 -> 6
- net /power_mgmt/powerpath_out: track 21.2 -> 27.7 mm
- net /power_mgmt/+5VUSB: track 19.2 -> 24.5 mm, vias 3 -> 2
- net Net-(U8-FB): track 4.11 -> 8.26 mm
- net /PREVGL: track 1.71 -> 5.67 mm
- net /GDR: track 4.56 -> 8.00 mm
- net /RESE: track 4.79 -> 7.91 mm
- net Net-(SSB43L1-K): track 14.7 -> 12.5 mm
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Other:
- board outline added: 38 x 32 mm

Commit message: Taseotlkauset
Parts:
- added C13: 1uf, Capacitor_SMD:C_0201_0603Metric, F.Cu at (158.7, 46.6)
- added C14: 0.1uf, Capacitor_SMD:C_0201_0603Metric, F.Cu at (163.2, 46.3)
- added SW2: K2-1109DE-D4SW-01, K2-1109DE-D4SW-01:KEY-TH_K2-1109DE-CXXW-XX, F.Cu at (139.2, 41.8)
- added U9: LTC2954CTS8-2_TRMPBF, LTC2954CTS8_2_TRMPBF:TSOT-23_TS8, F.Cu at (161.0, 45.8)
- FPC1: value FPC-05F-24PH20 -> AFC07-S24ECA-00; footprint FPC-05F-24PH20:FPC-SMD_24P-P0.50_FPC-05F-24PH20 -> FPC-SMD_AFC07-S24ECA-00:FPC-SMD_AFC07-S24ECA-00
- moved R15 1.27 mm to (151.8, 69.0)
- moved C10 0.75 mm to (162.5, 54.0)
- moved C11 0.75 mm to (160.8, 54.0)
- moved C12 0.75 mm to (160.8, 55.0)
- moved C9 0.75 mm to (166.8, 50.7)
- moved L1 0.75 mm to (160.8, 58.2)
- moved R11 0.75 mm to (159.2, 54.0)
- moved R12 0.75 mm to (159.2, 55.0)
- moved R13 0.75 mm to (166.8, 49.1)
- moved U8 0.75 mm to (162.5, 50.5)
- moved SSB43L1 0.65 mm to (165.3, 56.9)
- moved U6 0.63 mm to (163.8, 63.3)
- moved R2 0.41 mm to (159.2, 61.1)
- moved C5 0.23 mm to (159.6, 64.6)
Connections:
- net /power_mgmt/V_battery renamed /VBattery
- SW1 pad 1: unconnected-(SW1-Pad1) -> /power_btn
- SW1 pad 2: unconnected-(SW1-Pad2) -> GND
- SW1 pad 3: unconnected-(SW1-Pad3) -> GND
- U5 pad 15: unconnected-(U5-SYSOFF-Pad15) -> /powerpath_enable
Routing:
- net /powerpath_enable: track 0.00 -> 30.6 mm, vias 0 -> 2
- net GND: track 116.3 -> 130.1 mm, vias 48 -> 50
- net /power_btn: track 0.00 -> 5.00 mm
- net +3.3V: track 24.1 -> 28.3 mm, vias 6 -> 8
- net /I2C_SDA: track 82.7 -> 84.7 mm
- net /PREVGL: track 5.67 -> 3.76 mm
- net /VBattery: track 15.6 -> 17.1 mm
- net /power_mgmt/powerpath_out: track 27.7 -> 26.4 mm
- net Net-(U9-PDT): track 0.00 -> 1.25 mm
- net Net-(U5-ISET): track 1.26 -> 2.45 mm
- net Net-(U8-FB): track 8.26 -> 7.33 mm
- net /I2C_SCL: track 90.7 -> 91.1 mm, vias 5 -> 4

Commit message: okay
Parts:
- added C15: 1uf, Capacitor_SMD:C_0201_0603Metric, F.Cu at (159.5, 47.4)
- added R18: 10k, Resistor_SMD:R_0201_0603Metric, F.Cu at (161.0, 47.4)
- added TP1: +RESET, TestPoint:TestPoint_Pad_1.0x1.0mm, F.Cu at (131.0, 65.0)
- added TP2: -RESET, TestPoint:TestPoint_Pad_1.0x1.0mm, F.Cu at (131.0, 67.0)
- added TP3: BOOT, TestPoint:TestPoint_Pad_1.0x1.0mm, F.Cu at (131.0, 69.5)
- moved C21 20.8 mm to (135.4, 43.1), turned to -90 degrees
- moved C22 18.8 mm to (141.8, 46.1), turned to -90 degrees
- moved L2 18.4 mm to (132.5, 42.8), turned to 180 degrees
- moved D4 16.3 mm to (138.8, 47.5), turned to 0 degrees
- moved R17 15.9 mm to (137.0, 59.8)
- moved R16 13.5 mm to (137.0, 59.0)
- moved D3 12.3 mm to (138.8, 45.0)
- moved C23 11.8 mm to (137.0, 58.2)
- moved Q1 11.1 mm to (140.3, 59.3), turned to 0 degrees
- moved C30 6.41 mm to (137.7, 49.1)
- moved D2 5.34 mm to (140.0, 51.5), turned to 90 degrees
- moved FPC1 5.15 mm to (133.9, 54.7)
- moved C29 4.87 mm to (137.7, 49.9)
- moved C28 3.32 mm to (137.7, 50.6)
- moved C24 2.93 mm to (137.7, 53.6)
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Connections:
- SW1 pad 1: /power_btn -> GND
- SW1 pad 2: GND -> /power_btn
- SW2 pad 1: unconnected-(SW2-Pad1) -> /menu_btn
- U1 pad 10: unconnected-(U1-IO6-Pad10) -> /dsp_dc
- U1 pad 11: unconnected-(U1-IO7-Pad11) -> /dsp_rst
- U1 pad 13: /dsp_rst -> unconnected-(U1-IO9-Pad13)
- U1 pad 14: /dsp_dc -> unconnected-(U1-IO10-Pad14)
- U1 pad 15: /dsp_cs -> unconnected-(U1-IO11-Pad15)
- U1 pad 16: /dsp_sclk -> unconnected-(U1-IO12-Pad16)
- U1 pad 17: /dsp_sdi -> unconnected-(U1-IO13-Pad17)
- U1 pad 36: unconnected-(U1-IO40-Pad36) -> /power_kill
- U1 pad 4: unconnected-(U1-IO0-Pad4) -> Net-(U1-IO0)
- U1 pad 45: unconnected-(U1-EN-Pad45) -> Net-(U1-EN)
- U1 pad 6: unconnected-(U1-IO2-Pad6) -> /menu_btn
- U1 pad 7: unconnected-(U1-IO3-Pad7) -> /dsp_sdi
- U1 pad 8: unconnected-(U1-IO4-Pad8) -> /dsp_sclk
- U1 pad 9: unconnected-(U1-IO5-Pad9) -> /dsp_cs
Routing:
- net /VBattery: track 17.1 -> 38.2 mm, vias 2 -> 4
- net /power_kill: track 0.00 -> 13.4 mm, vias 0 -> 2
- net /I2C_SCL: track 91.1 -> 78.0 mm
- net /menu_btn: track 0.00 -> 12.0 mm, vias 0 -> 1
- net /I2C_SDA: track 84.7 -> 75.5 mm
- net /dsp_sdi: track 0.00 -> 8.70 mm
- net /dsp_sclk: track 0.00 -> 8.57 mm
- net /dsp_cs: track 0.00 -> 8.46 mm
- net /dsp_busy: track 0.00 -> 8.41 mm
- net /dsp_dc: track 0.00 -> 8.33 mm
- net /dsp_rst: track 0.00 -> 8.29 mm
- net GND: track 130.1 -> 138.0 mm, vias 50 -> 54
- net Net-(D4-A): track 20.1 -> 26.6 mm, vias 0 -> 3
- net /PREVGL: track 3.76 -> 9.57 mm, vias 0 -> 2
- net /USB-: track 22.2 -> 17.2 mm
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Other:
- outline, holes or cut-outs redrawn

Commit message: idk
Parts:
- added R19: 10k, Resistor_SMD:R_0201_0603Metric, F.Cu at (152.6, 65.8)
- added R20: 10k, Resistor_SMD:R_0201_0603Metric, F.Cu at (152.8, 64.7)
- added RST1: +RESET, TestPoint:TestPoint_Pad_2.0x2.0mm, F.Cu at (150.8, 49.5)
- moved TP1 5.14 mm to (131.0, 70.1)
- moved TP3 4.11 mm to (131.0, 65.4)
- moved C7 1.18 mm to (151.8, 64.7)
- moved TP2 0.79 mm to (131.0, 67.8)
- moved J3 0.39 mm to (138.6, 67.2)
- moved SW1 0.05 mm to (161.0, 41.7)
Connections:
- U4 pad 10: unconnected-(U4-BIN-Pad10) -> Net-(U4-BIN)
- U4 pad 12: unconnected-(U4-GPOUT-Pad12) -> Net-(U4-GPOUT)
- U4 pad 13: unconnected-(U4-PAD-Pad13) -> GND
Routing:
- net Net-(U1-EN): track 4.20 -> 44.9 mm, vias 0 -> 2
- net Net-(U1-IO0): track 0.00 -> 28.2 mm, vias 0 -> 2
- net Net-(U4-BIN): track 0.00 -> 1.16 mm
- net Net-(U4-GPOUT): track 0.00 -> 1.15 mm
- net /VBattery: track 38.2 -> 37.0 mm
- net /power_mgmt/battery_in: track 19.1 -> 19.6 mm
Other:
- board size 38 x 32 mm -> 40 x 32 mm
- board text added: "This is my electrisity circuit board"

Commit message: asejkthas
Parts:
- C1, C10, C11, C12, C13, C15, C2, C21, C22, C23, C24, C25, C26, C27, C28, C29, C3, C30, C4, C5, C6, C7, C8, C9: footprint Capacitor_SMD:C_0201_0603Metric -> Capacitor_SMD:C_0402_1005Metric
- R1, R10, R11, R12, R13, R14, R15, R16, R17, R19, R2, R20, R3, R4, R5, R6, R7, R8, R9: footprint Resistor_SMD:R_0201_0603Metric -> Resistor_SMD:R_0402_1005Metric
- moved C30 4.93 mm to (134.0, 45.8), turned to 0 degrees
- moved C10 4.67 mm to (166.8, 52.3)
- moved R12 2.38 mm to (161.2, 53.8)
- moved C7 1.95 mm to (152.3, 62.8), turned to -90 degrees
- moved C12 1.68 mm to (159.2, 54.7)
- moved R2 1.57 mm to (160.6, 60.3), turned to 0 degrees
- moved R13 1.40 mm to (166.8, 47.7)
- moved R19 1.30 mm to (151.9, 64.7), turned to -90 degrees
- moved R6 1.16 mm to (158.7, 70.7)
- moved C11 1.11 mm to (161.7, 54.7), turned to 180 degrees
- moved FPC1 1.08 mm to (133.9, 55.8)
- moved R17 1.01 mm to (137.4, 60.8)
- moved C9 0.98 mm to (166.8, 49.8), turned to 90 degrees
- moved C8 0.93 mm to (159.5, 63.0)
- moved L1 0.79 mm to (160.5, 57.5), turned to 90 degrees
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Routing:
- net /power_mgmt/+5VUSB: track 27.9 -> 21.4 mm
- net +3.3V: track 25.4 -> 30.9 mm, vias 9 -> 10
- net /RESE: track 10.3 -> 5.01 mm, vias 2 -> 0
- net Net-(SSB43L1-K): track 12.5 -> 17.2 mm
- net /VBattery: track 37.0 -> 33.6 mm, vias 4 -> 3
- net /USB-: track 17.2 -> 20.0 mm
- net Net-(C30-Pad2): track 2.27 -> 4.82 mm
- net /GDR: track 5.40 -> 7.93 mm
- net /USB+: track 22.1 -> 19.8 mm
- net Net-(U4-GPOUT): track 1.15 -> 3.23 mm
- net /PREVGL: track 9.57 -> 7.57 mm, vias 2 -> 0
- net /power_mgmt/battery_in: track 19.6 -> 21.3 mm
- net /I2C_SDA: track 75.5 -> 73.8 mm
- net Net-(U8-BST): track 3.88 -> 2.18 mm
- net GND: track 137.9 -> 139.2 mm, vias 54 -> 55
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
Commit message: laout
Parts:
- removed RST1: +RESET, TestPoint:TestPoint_Pad_2.0x2.0mm
- C14: footprint Capacitor_SMD:C_0201_0603Metric -> Capacitor_SMD:C_0402_1005Metric
- R18: footprint Resistor_SMD:R_0201_0603Metric -> Resistor_SMD:R_0402_1005Metric
- moved R18 24.2 mm to (141.6, 61.9), turned to -90 degrees
- moved C14 1.52 mm to (164.5, 47.3)
- moved C13 0.76 mm to (158.9, 45.2), turned to 90 degrees
- moved D2 0.63 mm to (139.9, 51.1)
- moved C6 0.61 mm to (143.7, 62.6), turned to 0 degrees
- moved R4 0.44 mm to (145.6, 62.6)
- moved C15 0.43 mm to (158.9, 47.1), turned to 90 degrees
- moved U9 0.37 mm to (161.5, 45.9)
Routing:
- net /powerpath_enable: track 31.1 -> 34.2 mm
- net /power_kill: track 13.4 -> 11.1 mm
- net Net-(J1-CC1): track 1.68 -> 0.00 mm
- net Net-(U1-EN): track 44.5 -> 43.1 mm, vias 2 -> 3
- net /VBattery: track 33.6 -> 34.4 mm
- net Net-(D2-A): track 7.60 -> 6.84 mm
- net GND: track 139.2 -> 139.4 mm, vias 55 -> 58

Commit message: this is an electricity PCB
Connections:
- FPC1 pad 16: unconnected-(FPC1-Pad16) -> +3.3V
- FPC1 pad 17: unconnected-(FPC1-Pad17) -> GND
- FPC1 pad 6: /I2C_SCL -> unconnected-(FPC1-Pad6)
- FPC1 pad 7: /I2C_SDA -> unconnected-(FPC1-Pad7)
- FPC1 pad 8: unconnected-(FPC1-Pad8) -> GND
- J3 pad 1: GND -> /power_mgmt/battery_in
- J3 pad 2: /power_mgmt/battery_in -> GND
- R9 pad 1: /power_mgmt/CHG -> /charging_status
- U1 pad 13: unconnected-(U1-IO9-Pad13) -> /clock_alarm
- U1 pad 28: unconnected-(U1-IO33-Pad28) -> /charging_status
- U1 pad 32: unconnected-(U1-IO36-Pad32) -> /btn_int
- U1 pad 33: unconnected-(U1-IO37-Pad33) -> /power_kill
- U1 pad 36: /power_kill -> unconnected-(U1-IO40-Pad36)
- U2 pad 3: unconnected-(U2-~{INT}/SQW-Pad3) -> /clock_alarm
- U5 pad 9: /power_mgmt/CHG -> /charging_status
Routing:
- net /clock_alarm: track 0.00 -> 31.6 mm, vias 0 -> 2
- net /I2C_SCL: track 78.1 -> 53.3 mm, vias 4 -> 2
- net /I2C_SDA: track 73.9 -> 49.4 mm, vias 6 -> 3
- net /btn_int: track 0.00 -> 18.9 mm, vias 0 -> 2
- net /charging_status: track 0.00 -> 14.4 mm, vias 0 -> 2
- net GND: track 139.4 -> 144.9 mm, vias 58 -> 59
- net /powerpath_enable: track 34.2 -> 30.1 mm
- net /power_kill: track 11.1 -> 13.7 mm
- net Net-(J1-CC1): track 0.00 -> 1.91 mm
- net Net-(U1-EN): track 43.1 -> 41.2 mm
- net +3.3V: track 31.3 -> 32.9 mm, vias 10 -> 11
- net /power_mgmt/powerpath_out: track 27.2 -> 25.7 mm
- net /power_mgmt/CHG: track 1.35 -> 0.00 mm
- net /power_mgmt/battery_in: track 21.3 -> 20.7 mm
