File: templog_mainboard/templog_mainboard.kicad_pcb (KiCad board)
At the start: 4 copper layers, 40 x 32 mm, 69 parts, among them J1 USB_C_Receptacle_USB2.0_16P, J3 battery_con, Q1 Si1308EDL, SW1 K2-1109DE-D4SW-01, SW2 K2-1109DE-D4SW-01, U1 ESP32-S3-MINI-1, U2 DS3231MZ, U3 SHT4x, U4 BQ27441-G1, U5 BQ24075RGT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

Commit message: ummmmmm uggg uhhh
Routing:
- net /VBattery: track 34.6 -> 33.8 mm
Changed lines of the file:
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@@
+	)
+	(segment
+		(start 154.079499 62.329499)
+		(end 154.383471 62.329499)
+		(width 0.25)
+		(layer "B.Cu")
+		(net 87)
+	)
+	(segment
+		(start 153.019358 58.673249)
+		(end 153.019358 61.269358)
+		(width 0.25)
+		(layer "B.Cu")
+		(net 87)
+	)
+	(segment
+		(start 162.638946 49.053661)
+		(end 153.019358 58.673249)
+		(width 0.25)
+		(layer "B.Cu")
+		(net 87)
+	)
+	(segment
+		(start 154.070643 62.642327)
+		(end 154.383471 62.329499)
+		(width 0.25)
+		(layer "B.Cu")
+		(net 87)
+	)
+	(segment
+		(start 162.638946 48.13548)
+		(end 162.638946 49.053661)
+		(width 0.25)
+		(layer "B.Cu")
+		(net 87)
+	)
+	(segment
+		(start 155.365376 70.95)
+		(end 154.070643 69.655267)
+		(width 0.25)
+		(layer "B.Cu")
+		(net 87)
+	)
+	(segment
+		(start 154.070643 69.655267)
+		(end 154.070643 62.642327)
+		(width 0.25)
+		(layer "B.Cu")
+		(net 87)
+	)
+	(segment
+		(start 153.019358 61.269358)
+		(end 154.079499 62.329499)
+		(width 0.25)
+		(layer "B.Cu")
+		(net 87)
 	)
 	(segment
 		(start 162.656349 48.118077)
 		(end 162.638946 48.13548)
-		(width 0.25)
-		(layer "B.Cu")
-		(net 87)
-	)
-	(segment
-		(start 154.079499 62.329499)
-		(end 154.383471 62.329499)
-		(width 0.25)
-		(layer "B.Cu")
-		(net 87)
-	)
-	(segment
-		(start 162.638946 48.13548)
-		(end 161.26263 48.13548)
-		(width 0.25)
-		(layer "B.Cu")
-		(net 87)
-	)
-	(segment
-		(start 154.070643 62.642327)
-		(end 154.383471 62.329499)
-		(width 0.25)
-		(layer "B.Cu")
-		(net 87)
-	)
-	(segment
-		(start 155.365376 70.95)
-		(end 154.070643 69.655267)
-		(width 0.25)
-		(layer "B.Cu")
-		(net 87)
-	)
-	(segment
-		(start 154.070643 69.655267)
-		(end 154.070643 62.642327)
-		(width 0.25)
-		(layer "B.Cu")
-		(net 87)
-	)
-	(segment
-		(start 161.26263 48.13548)
-		(end 153.019358 56.378752)
-		(width 0.25)
-		(layer "B.Cu")
-		(net 87)
-	)
-	(segment
-		(start 153.019358 61.269358)
-		(end 154.079499 62.329499)
-		(width 0.25)
-		(layer "B.Cu")
-		(net 87)
-	)
-	(segment
-		(start 153.019358 56.378752)
-		(end 153.019358 61.269358)
 		(width 0.25)
 		(layer "B.Cu")
@@
 	)
 	(segment
-		(start 152 56.645243)
-		(end 152 62)
-		(width 0.25)
-		(layer "B.Cu")
-		(net 89)
-	)
-	(segment
 		(start 152 62)
 		(end 153.411903 63.411903)
@@
 	)
 	(segment
+		(start 153.411903 69.030039)
+		(end 153.316942 69.125)
+		(width 0.25)
+		(layer "B.Cu")
+		(net 89)
+	)
+	(segment
+		(start 161.433567 47.493162)
+		(end 161.433567 47.816433)
+		(width 0.25)
+		(layer "B.Cu")
+		(net 89)
+	)
+	(segment
+		(start 152 57.25)
+		(end 152 62)
+		(width 0.25)
+		(layer "B.Cu")
+		(net 89)
+	)
+	(segment
 		(start 153.411903 63.411903)
 		(end 153.411903 69.030039)
@@
 	)
 	(segment
-		(start 161.152081 47.493162)
-		(end 152 56.645243)
-		(width 0.25)
-		(layer "B.Cu")
-		(net 89)
-	)
-	(segment
-		(start 153.411903 69.030039)
-		(end 153.316942 69.125)
-		(width 0.25)
-		(layer "B.Cu")
-		(net 89)
-	)
-	(segment
-		(start 161.433567 47.493162)
-		(end 161.152081 47.493162)
-		(width 0.25)
-		(layer "B.Cu")
+		(start 161.433567 47.816433)
+		(end 152 57.25)
+		(width 0.25)
+		(layer "B.Cu")

Commit message: electroscity
Parts:
- C2: footprint Capacitor_SMD:C_0402_1005Metric -> Capacitor_SMD:C_0603_1608Metric
- moved R9 3.81 mm to (156.3, 62.4), turned to 180 degrees
- moved R19 1.05 mm to (152.7, 65.5), turned to 0 degrees
- moved R14 0.81 mm to (152.7, 66.5)
- moved U4 0.81 mm to (156.3, 64.7)
- moved R20 0.73 mm to (152.7, 64.4), turned to 180 degrees
- moved C2 0.52 mm to (141.5, 51.2)
- moved D2 0.24 mm to (139.6, 51.1)
- moved C7 0.13 mm to (152.3, 63.0)
- moved R5 0.10 mm to (153.3, 62.9)
Connections:
- R9 pad 1: /charging_status -> +3.3V
- R9 pad 2: +3.3V -> /clock_alarm
- U1 pad 13: /clock_alarm -> unconnected-(U1-IO9-Pad13)
- U1 pad 25: unconnected-(U1-IO21-Pad25) -> /clock_alarm
Routing:
- net /clock_alarm: track 31.6 -> 23.3 mm
- net /charging_status: track 14.4 -> 11.6 mm
- net Net-(U4-GPOUT): track 3.23 -> 1.31 mm
- net GND: track 144.9 -> 146.8 mm, vias 59 -> 60
- net /power_mgmt/battery_in: track 20.7 -> 22.1 mm, vias 1 -> 2
- net /power_mgmt/powerpath_out: track 25.7 -> 26.9 mm
- net /I2C_SCL: track 53.3 -> 52.4 mm
- net /I2C_SDA: track 49.4 -> 48.6 mm
- net Net-(U5-ILIM): track 1.47 -> 2.17 mm
- net Net-(U4-V_{DD}): track 1.11 -> 1.79 mm
- net /powerpath_enable: track 29.9 -> 29.3 mm

Commit message: :ASEDfasef
Parts:
- removed C11, C12: 47uf, Capacitor_SMD:C_0402_1005Metric
- removed R11, R12: 31.6k, Resistor_SMD:R_0402_1005Metric
- removed R13: 100k, Resistor_SMD:R_0402_1005Metric
- removed SSB43L1: D, Diode_SMD:D_SMB
- C10: value 0.1uf -> 10uf; footprint Capacitor_SMD:C_0402_1005Metric -> Capacitor_SMD:C_0805_2012Metric
- C2: footprint Capacitor_SMD:C_0603_1608Metric -> Capacitor_SMD:C_0805_2012Metric
- C21, C22: footprint Capacitor_SMD:C_0402_1005Metric -> Capacitor_SMD:C_0603_1608Metric
- C9: footprint Capacitor_SMD:C_0402_1005Metric -> Capacitor_SMD:C_0805_2012Metric
- L1: value 4.7uH -> 10uH
- U8: value ADP2303ARDZ-3.3 -> TPS62203DBV; footprint Package_SO:SOIC-8-1EP_3.9x4.9mm_P1.27mm_EP2.29x3mm -> Package_TO_SOT_SMD:SOT-23-5
- moved C9 10.1 mm to (159.8, 57.1), turned to -90 degrees
- moved U8 6.98 mm to (162.5, 57.5), turned to 90 degrees
- moved C10 5.43 mm to (165.3, 57.5), turned to 90 degrees
- moved C13 4.53 mm to (159.5, 49.7), turned to -90 degrees
- moved L1 4.48 mm to (161.2, 53.1), turned to 0 degrees
- moved U9 2.60 mm to (162.1, 48.4)
- moved C14 1.38 mm to (164.8, 48.6), turned to 90 degrees
- moved R2 0.87 mm to (161.4, 60.1)
- moved C1 0.78 mm to (142.0, 47.9)
- moved C22 0.76 mm to (141.9, 45.3)
- moved C15 0.73 mm to (159.5, 47.5)
- moved U1 0.43 mm to (150.7, 51.3)
- moved R1 0.41 mm to (159.5, 61.1), turned to 90 degrees
- moved D2 0.15 mm to (139.5, 51.1)
- moved C2 0.13 mm to (141.7, 51.2)
Connections:
- C10 pad 1: Net-(U8-BST) -> GND
- C10 pad 2: Net-(SSB43L1-K) -> +3.3V
- L1 pad 1: Net-(SSB43L1-K) -> Net-(U8-SW)
- U8 pad 1: Net-(U8-BST) -> /power_mgmt/powerpath_out
- U8 pad 2: /power_mgmt/powerpath_out -> GND
- U8 pad 4: Net-(U8-PGOOD) -> +3.3V
- U8 pad 5: Net-(U8-FB) -> Net-(U8-SW)
Routing:
- net Net-(SSB43L1-K): track 17.2 -> 0.00 mm
- net /power_mgmt/powerpath_out: track 26.9 -> 16.2 mm
- net GND: track 146.8 -> 137.8 mm, vias 60 -> 58
- net Net-(U8-FB): track 7.32 -> 0.00 mm
- net /power_btn: track 5.56 -> 8.54 mm
- net Net-(U8-SW): track 0.00 -> 2.56 mm
- net Net-(U8-PGOOD): track 2.37 -> 0.00 mm
- net /powerpath_enable: track 29.3 -> 27.0 mm
- net Net-(U8-BST): track 2.18 -> 0.00 mm
- net /VBattery: track 33.9 -> 31.7 mm
- net /I2C_SDA: track 48.6 -> 50.6 mm
- net Net-(U1-IO0): track 28.4 -> 26.7 mm
- net /btn_int: track 18.9 -> 17.2 mm
- net +3.3V: track 33.1 -> 32.4 mm
- net /power_kill: track 13.7 -> 13.1 mm
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Other:
- outline, holes or cut-outs redrawn

Commit message: electractiyt
Parts:
- added G***: LOGO, LOGO, F.Cu at (165.5, 52.8)
- C13, C23, C24, C25, C26, C27, C28, C29, C30, C6: footprint Capacitor_SMD:C_0402_1005Metric -> Capacitor_SMD:C_0603_1608Metric
- moved R18 24.5 mm to (159.6, 45.2), turned to 0 degrees
- moved R16 5.61 mm to (142.2, 62.3), turned to 90 degrees
- moved C25 4.71 mm to (142.0, 54.4), turned to -90 degrees
- moved C29 4.31 mm to (134.9, 45.8), turned to 0 degrees
- moved R17 3.76 mm to (140.8, 62.3), turned to 90 degrees
- moved C26 2.77 mm to (139.6, 53.9)
- moved C24 2.63 mm to (139.6, 55.7)
- moved C30 2.39 mm to (131.6, 45.8)
- moved C23 1.95 mm to (137.8, 60.1)
- moved C27 1.69 mm to (137.4, 53.0), turned to 90 degrees
- moved R4 1.57 mm to (144.8, 63.9)
- moved C15 1.30 mm to (159.6, 46.2), turned to 180 degrees
- moved J1 1.21 mm to (145.8, 69.2)
- moved Q1 1.01 mm to (141.0, 60.0), turned to 180 degrees
- moved R3 0.84 mm to (150.0, 63.4), turned to 90 degrees
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Connections:
- U1 pad 10: /dsp_dc -> /dsp_sdi
- U1 pad 11: /dsp_rst -> /dsp_sclk
- U1 pad 12: /dsp_busy -> /dsp_cs
- U1 pad 13: unconnected-(U1-IO9-Pad13) -> /dsp_dc
- U1 pad 14: unconnected-(U1-IO10-Pad14) -> /dsp_rst
- U1 pad 15: unconnected-(U1-IO11-Pad15) -> /dsp_busy
- U1 pad 7: /dsp_sdi -> unconnected-(U1-IO3-Pad7)
- U1 pad 8: /dsp_sclk -> unconnected-(U1-IO4-Pad8)
- U1 pad 9: /dsp_cs -> unconnected-(U1-IO5-Pad9)
- U7 pad 2: /power_mgmt/+5VUSB -> GND
- U7 pad 3: unconnected-(U7-I/O2-Pad3) -> /USB+
- U7 pad 5: GND -> /power_mgmt/+5VUSB
- U7 pad 6: /USB+ -> unconnected-(U7-I/O1-Pad6)
Routing:
- net Net-(C25-Pad2): track 1.87 -> 11.0 mm, vias 0 -> 2
- net /RESE: track 5.01 -> 10.4 mm
- net /power_mgmt/powerpath_out: track 16.2 -> 19.4 mm
- net +3.3V: track 32.4 -> 35.3 mm
- net Net-(C26-Pad2): track 1.85 -> 4.47 mm
- net Net-(C24-Pad2): track 1.80 -> 4.26 mm
- net /power_mgmt/battery_in: track 22.1 -> 24.2 mm
- net Net-(U1-EN): track 41.7 -> 43.7 mm, vias 3 -> 2
- net /USB+: track 20.3 -> 22.2 mm
- net /dsp_busy: track 7.73 -> 9.62 mm
- net Net-(J1-CC2): track 2.37 -> 3.79 mm
- net Net-(C30-Pad2): track 4.62 -> 6.04 mm
- net /btn_int: track 17.2 -> 18.6 mm
- net /dsp_rst: track 8.30 -> 9.32 mm
- net Net-(D4-A): track 26.9 -> 27.7 mm
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Other:
- outline, holes or cut-outs redrawn

Commit message: uuhhuh umm electriciadty
Parts:
- moved R5 0.89 mm to (152.7, 62.4), turned to 0 degrees
- moved C7 0.57 mm to (152.7, 63.4), turned to 0 degrees
- moved U4 0.20 mm to (156.3, 64.9)
Routing:
- net /power_mgmt/battery_in: track 24.2 -> 29.3 mm
- net GND: track 138.3 -> 136.2 mm, vias 62 -> 63
- net /VBattery: track 31.6 -> 29.8 mm
- net /clock_alarm: track 22.9 -> 22.2 mm
- net /power_mgmt/powerpath_out: track 19.4 -> 18.9 mm
- net +3.3V: vias 11 -> 12
