File: templog_mainboard/power_mgmt.kicad_sch (KiCad schematic)
At the start: 2 parts, among them U4 BQ27441-G1, U5 BQ24075RGT

Commit message: elecricity
Parts:
- added C6: 4.7uf, Capacitor_SMD:C_0201_0603Metric, symbol Device:C
- added C7: 1.0uf, Capacitor_SMD:C_0201_0603Metric, symbol Device:C
- added C8: 0.47uf, Capacitor_SMD:C_0201_0603Metric, symbol Device:C
- added J1: USB_C_Receptacle_USB2.0_16P, Connector_USB:USB_C_Receptacle_GCT_USB4105-xx-A_16P_TopMnt_Horizontal, symbol Connector:USB_C_Receptacle_USB2.0_16P
- added J3: battery_con, Connector_JST:JST_PH_S2B-PH-K_1x02_P2.00mm_Horizontal, symbol Connector_Generic:Conn_01x02
- added R10, R7, R8, R9: 10k, Resistor_SMD:R_0201_0603Metric, symbol Device:R_US
- added R3, R4: 5.1k, Resistor_SMD:R_0201_0603Metric, symbol Device:R_US
- added R5: 0.01, Resistor_SMD:R_0201_0603Metric, symbol Device:R_US
- added R6: 100k, Resistor_SMD:R_0201_0603Metric, symbol Device:R_US
- added U7: USBLC6-2SC6, Package_TO_SOT_SMD:SOT-23-6, symbol Power_Protection:USBLC6-2SC6
- added U8: ADP2303ARDZ-3.3, Package_SO:SOIC-8-1EP_3.9x4.9mm_P1.27mm_EP2.29x3mm, symbol Regulator_Switching:ADP2303ARDZ-3.3
Connections:
- net ESP_SDA: now reaches U4.1 (SDA)
- net ESP_SCL: now reaches U4.2 (SCL)
- net GND: now reaches U4.3 (V_{SS})
- net GND: now also U5.17 (VSS), U5.8 (VSS), C6.2, C7.1, C8.1, J1.A1 (GND), J1.A12 (GND), J1.B1 (GND), J1.B12 (GND), J3.1 (Pin_1), R10.2, R3.2, R4.2, R6.1, R7.1, R8.1, U7.5 (VBUS), U8.7 (GND)
- net at U4.5 (V_{DD}): now also C8.2
- net battery_in: now reaches U4.6 (BAT)
- net battery_in: now also U4.8 (SRP), C7.2, J3.2 (Pin_2), R5.1
- net V_battery: now reaches U4.7 (SRN)
- net V_battery: now also U5.2 (BAT), U5.3 (BAT), R5.2
- net at U5.1 (TS): now also R10.1
- net powerpath_out: now reaches U5.10 (OUT), U5.11 (OUT)
- net powerpath_out: now also U8.2 (Vin)
- net +5VUSB: now reaches U5.13 (IN)
- net +5VUSB: now also C6.1, J1.A4 (VBUS), J1.A9 (VBUS), J1.B4 (VBUS), J1.B9 (VBUS), U7.2 (GND)
- net at U5.4 (~{CE}): now also R6.2
- net at U5.5 (EN2): now also R8.2
- net at U5.6 (EN1): now also R7.2
- net CHG: now reaches U5.9 (~{CHG})
- net CHG: now also R9.1
- new net: J1.A5 (CC1), R4.1
- new net: J1.B5 (CC2), R3.1
- new net +3.3Vout: R9.2
- new net USB_D-: J1.A7 (D-), J1.B7 (D-), U7.4 (I/O2), U7.6 (I/O1)
- new net USB_d+: J1.A6 (D+), J1.B6 (D+)
- no-connect marks 0 -> 6
Other:
- moved on the sheet: U4, U5

Commit message: electtrirciy
Parts:
- added C10: 0.1uf, Capacitor_SMD:C_0201_0603Metric, symbol Device:C
- added C11, C12: 47uf, Capacitor_SMD:C_0201_0603Metric, symbol Device:C
- added C9: 10uf, Capacitor_SMD:C_0201_0603Metric, symbol Device:C
- added D1: D, Diode_SMD:D_0201_0603Metric, symbol Device:D
- added L1: 4.7uH, Inductor_SMD:L_6.3x6.3_H3, symbol Device:L
- added R11, R12: 31.6k, Resistor_SMD:R_0201_0603Metric, symbol Device:R_US
- added R13: 100k, Resistor_SMD:R_0201_0603Metric, symbol Device:R_US
- added R14, R15: 2.2k, Resistor_SMD:R_0201_0603Metric, symbol Device:R_US
Connections:
- net +3.3Vout: now also C11.1, C12.1, L1.2, R11.1
- net GND: now also U5.14 (TMR), C9.1, D1.2 (A), R12.2, R14.1, R15.1
- net USB_D-: no longer U7.6 (I/O1)
- net USB_d+: now also U7.6 (I/O1)
- net powerpath_out: now also U8.3 (EN), C9.2, R13.1
- net at U5.12 (ILIM): now also R14.2
- net at U5.16 (ISET): now also R15.2
- net at U8.1 (BST): now also C10.1
- net at U8.4 (PGOOD): now also R13.2
- net at U8.5 (FB): now also R11.2, R12.1
- net at U8.8 (SW): now also C10.2, D1.1 (K), L1.1
Other:
- moved on the sheet: R10, R6, R7, R8, R9, U5, U8

Commit message: time for electricity
Parts:
- L1: footprint Inductor_SMD:L_6.3x6.3_H3 -> Inductor_SMD:L_Sunlord_SWPA4030S
- SSB43L1: renamed from D1; footprint Diode_SMD:D_0201_0603Metric -> Diode_SMD:D_SMB
Connections:
- net GND: now also C11.2, C12.2
Changed lines of the file:
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@@
 	)
 	(junction
-		(at 250.19 106.68)
-		(diameter 0)
-		(color 0 0 0 0)
-	)
-	(junction
 		(at 60.96 88.9)
 		(diameter 0)
@@
 	)
 	(junction
+		(at 250.19 107.95)
+		(diameter 0)
+		(color 0 0 0 0)
+	)
+	(junction
 		(at 90.17 132.08)
 		(diameter 0)
@@
 	(wire
 		(pts
-			(xy 200.66 100.33) (xy 200.66 118.11)
+			(xy 250.19 102.87) (xy 250.19 107.95)
 		)
 		(stroke
@@
 	(wire
 		(pts
-			(xy 261.62 95.25) (xy 261.62 99.06)
+			(xy 200.66 100.33) (xy 200.66 118.11)
 		)
 		(stroke
@@
 	(wire
 		(pts
-			(xy 46.99 33.02) (xy 50.8 33.02)
+			(xy 261.62 95.25) (xy 261.62 99.06)
 		)
 		(stroke
@@
 	(wire
 		(pts
-			(xy 250.19 102.87) (xy 250.19 106.68)
+			(xy 46.99 33.02) (xy 50.8 33.02)
 		)
 		(stroke
@@
 	(wire
 		(pts
-			(xy 250.19 106.68) (xy 250.19 107.95)
-		)
-		(stroke
-			(width 0)
-			(type default)
-		)
-	)
-	(wire
-		(pts
 			(xy 250.19 95.25) (xy 261.62 95.25)
 		)
@@
 	(wire
 		(pts
+			(xy 238.76 102.87) (xy 238.76 104.14)
+		)
+		(stroke
+			(width 0)
+			(type default)
+		)
+	)
+	(wire
+		(pts
 			(xy 152.4 100.33) (xy 171.45 100.33)
 		)
@@
 	(wire
 		(pts
+			(xy 227.33 102.87) (xy 227.33 104.14)
+		)
+		(stroke
+			(width 0)
+			(type default)
+		)
+	)
+	(wire
+		(pts
 			(xy 123.19 36.83) (xy 123.19 40.64)
 		)
@@
 	(wire
 		(pts
-			(xy 215.9 118.11) (xy 215.9 106.68)
+			(xy 215.9 118.11) (xy 215.9 107.95)
 		)
 		(stroke
@@
 	(wire
 		(pts
-			(xy 215.9 106.68) (xy 250.19 106.68)
+			(xy 215.9 107.95) (xy 250.19 107.95)
 		)
 		(stroke
@@
 	)
 	(symbol
+		(lib_id "power:GND")
+		(at 238.76 104.14 0)
+		(unit 1)
+		(exclude_from_sim no)
+		(in_bom yes)
+		(on_board yes)
+		(dnp no)
+		(fields_autoplaced yes)
+		(property "Reference" "#PWR033"
+			(at 238.76 110.49 0)
+			(effects
+				(font
+					(size 1.27 1.27)
+				)
+				(hide yes)
+			)
+		)
+		(property "Value" "GND"
+			(at 238.76 109.22 0)
+			(effects
+				(font
+					(size 1.27 1.27)
+				)
+			)
+		)
+		(property "Footprint" ""
+			(at 238.76 104.14 0)
+			(effects
+				(font
+					(size 1.27 1.27)
+				)
+				(hide yes)
+			)
+		)
+		(property "Datasheet" ""
+			(at 238.76 104.14 0)
+			(effects
+				(font
+					(size 1.27 1.27)
+				)
+				(hide yes)
+			)
+		)
+		(property "Description" "Power symbol creates a global label with name \"GND\" , ground"
+			(at 238.76 104.14 0)
+			(effects
+				(font
+					(size 1.27 1.27)
+				)
+				(hide yes)
+			)
+		)
+		(pin "1"
+		)
+		(instances
+			(project "templog_mainboard"
+				(path "/84b25dc3-cc11-42e1-888d-24c6d5a62713/d593db04-482a-483f-ba64-3cc83809d23e"
+					(reference "#PWR033")
+					(unit 1)
+				)
+			)
+		)
+	)
+	(symbol
 		(lib_id "Device:C")
 		(at 123.19 33.02 0)
@@
 		(dnp no)
 		(fields_autoplaced yes)
-		(property "Reference" "D1"
+		(property "Reference" "SSB43L1"
 			(at 209.55 100.3299 90)
 			(effects
@@
 			)
 		)
-		(property "Footprint" "Diode_SMD:D_0201_0603Metric"
+		(property "Footprint" "Diode_SMD:D_SMB"
 			(at 207.01 101.6 0)
 			(effects
@@
 			(project ""
 				(path "/84b25dc3-cc11-42e1-888d-24c6d5a62713/d593db04-482a-483f-ba64-3cc83809d23e"
-					(reference "D1")
+					(reference "SSB43L1")
 					(unit 1)
 				)
@@
 	(symbol
 		(lib_id "power:GND")
+		(at 227.33 104.14 0)
+		(unit 1)
+		(exclude_from_sim no)
+		(in_bom yes)
+		(on_board yes)
+		(dnp no)
+		(fields_autoplaced yes)
+		(property "Reference" "#PWR034"
+			(at 227.33 110.49 0)
+			(effects
+				(font
+					(size 1.27 1.27)
+				)
+				(hide yes)
+			)
+		)
+		(property "Value" "GND"
+			(at 227.33 109.22 0)
+			(effects
+				(font
+					(size 1.27 1.27)
+				)
+			)
+		)
+		(property "Footprint" ""
+			(at 227.33 104.14 0)
+			(effects
+				(font
+					(size 1.27 1.27)
+				)
+				(hide yes)
+			)
+		)
+		(property "Datasheet" ""
+			(at 227.33 104.14 0)
+			(effects
+				(font
+					(size 1.27 1.27)
+				)
+				(hide yes)
+			)
+		)
+		(property "Description" "Power symbol creates a global label with name \"GND\" , ground"
+			(at 227.33 104.14 0)
+			(effects
+				(font
+					(size 1.27 1.27)
+				)
+				(hide yes)
+			)
+		)
+		(pin "1"
+		)
+		(instances
+			(project "templog_mainboard"
+				(path "/84b25dc3-cc11-42e1-888d-24c6d5a62713/d593db04-482a-483f-ba64-3cc83809d23e"
+					(reference "#PWR034")
+					(unit 1)
+				)
+			)
+		)
+	)
+	(symbol
+		(lib_id "power:GND")
 		(at 123.19 25.4 180)
 		(unit 1)
@@
 			)
 		)
-		(property "Footprint" "Inductor_SMD:L_6.3x6.3_H3"
+		(property "Footprint" "Inductor_SMD:L_Sunlord_SWPA4030S"
 			(at 220.98 95.25 0)
 			(effects

Commit message: Taseotlkauset
Connections:
- net SYSOFF: now reaches U5.15 (SYSOFF)
- net V_battery renamed +battery
Changed lines of the file:
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@@
+	(wire
+		(pts
+			(xy 74.93 41.91) (xy 80.01 41.91)
+		)
+		(stroke
+			(width 0)
+			(type default)
+		)
+	)
 	(wire
 		(pts
@@
 	(wire
 		(pts
+			(xy 111.76 116.84) (xy 114.3 116.84)
+		)
+		(stroke
+			(width 0)
+			(type default)
+		)
+	)
+	(wire
+		(pts
 			(xy 196.85 100.33) (xy 200.66 100.33)
 		)
@@
 		(pts
 			(xy 144.78 66.04) (xy 144.78 69.85)
+		)
+		(stroke
+			(width 0)
+			(type default)
+		)
+	)
+	(wire
+		(pts
+			(xy 111.76 109.22) (xy 111.76 116.84)
 		)
 		(stroke
@@
 			)
 			(justify left bottom)
+		)
+	)
+	(label "V_battery"
+		(at 74.93 41.91 180)
+		(effects
+			(font
+				(size 1.27 1.27)
+			)
+			(justify right bottom)
 		)
 	)
@@
 		)
 	)
+	(hierarchical_label "+battery"
+		(shape output)
+		(at 80.01 41.91 0)
+		(effects
+			(font
+				(size 1.27 1.27)
+			)
+			(justify left)
+		)
+	)
 	(hierarchical_label "ESP_SCL"
 		(shape output)
@@
 		(effects
 			(font
+				(size 1.27 1.27)
+			)
+			(justify left)
+		)
+	)
+	(hierarchical_label "SYSOFF"
+		(shape input)
+		(at 111.76 109.22 90)
+		(effects
+			(font

Commit message: idk
Parts:
- added R19, R20: 10k, Resistor_SMD:R_0201_0603Metric, symbol Device:R_US
Connections:
- net GND: now also U4.13 (PAD), R20.2
- net battery_in: now also R19.1
- net at U4.10 (BIN): now also R20.1
- net at U4.12 (GPOUT): now also R19.2
Other:
- moved on the sheet: C10, C11, C12, C6, C7, C8, C9, J1, J3, L1, R10, R11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

Commit message: asejkthas
Parts:
- C10, C11, C12, C6, C7, C8, C9: footprint Capacitor_SMD:C_0201_0603Metric -> Capacitor_SMD:C_0402_1005Metric
- R10, R11, R12, R13, R14, R15, R19, R20, R3, R4, R5, R6, R7, R8, R9: footprint Resistor_SMD:R_0201_0603Metric -> Resistor_SMD:R_0402_1005Metric
Changed lines of the file:
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@@
 			)
 		)
-		(property "Footprint" "Resistor_SMD:R_0201_0603Metric"
+		(property "Footprint" "Resistor_SMD:R_0402_1005Metric"
 			(at 153.416 113.284 90)
 			(effects
@@
 			)
 		)
-		(property "Footprint" "Resistor_SMD:R_0201_0603Metric"
+		(property "Footprint" "Resistor_SMD:R_0402_1005Metric"
 			(at 67.564 73.914 90)
 			(effects
@@
 			)
 		)
-		(property "Footprint" "Capacitor_SMD:C_0201_0603Metric"
+		(property "Footprint" "Capacitor_SMD:C_0402_1005Metric"
 			(at 228.2952 120.65 0)
 			(effects
@@
 			)
 		)
-		(property "Footprint" "Capacitor_SMD:C_0201_0603Metric"
+		(property "Footprint" "Capacitor_SMD:C_0402_1005Metric"
 			(at 105.1052 35.56 0)
 			(effects
@@
 			)
 		)
-		(property "Footprint" "Capacitor_SMD:C_0201_0603Metric"
+		(property "Footprint" "Capacitor_SMD:C_0402_1005Metric"
 			(at 144.78 42.8752 0)
 			(effects
@@
 			)
 		)
-		(property "Footprint" "Resistor_SMD:R_0201_0603Metric"
+		(property "Footprint" "Resistor_SMD:R_0402_1005Metric"
 			(at 251.206 117.094 90)
 			(effects
@@
 			)
 		)
-		(property "Footprint" "Capacitor_SMD:C_0201_0603Metric"
+		(property "Footprint" "Capacitor_SMD:C_0402_1005Metric"
 			(at 43.18 120.3452 0)
 			(effects
@@
 			)
 		)
-		(property "Footprint" "Resistor_SMD:R_0201_0603Metric"
+		(property "Footprint" "Resistor_SMD:R_0402_1005Metric"
 			(at 67.564 82.804 90)
 			(effects
@@
 			)
 		)
-		(property "Footprint" "Resistor_SMD:R_0201_0603Metric"
+		(property "Footprint" "Resistor_SMD:R_0402_1005Metric"
 			(at 251.206 129.794 90)
 			(effects
@@
 			)
 		)
-		(property "Footprint" "Resistor_SMD:R_0201_0603Metric"
+		(property "Footprint" "Resistor_SMD:R_0402_1005Metric"
 			(at 96.774 51.054 90)
 			(effects
@@
 			)
 		)
-		(property "Footprint" "Resistor_SMD:R_0201_0603Metric"
+		(property "Footprint" "Resistor_SMD:R_0402_1005Metric"
 			(at 87.884 150.114 90)
 			(effects
@@
 			)
 		)
-		(property "Footprint" "Resistor_SMD:R_0201_0603Metric"
+		(property "Footprint" "Resistor_SMD:R_0402_1005Metric"
 			(at 94.234 162.306 90)
 			(effects
@@
 			)
 		)
-		(property "Footprint" "Capacitor_SMD:C_0201_0603Metric"
+		(property "Footprint" "Capacitor_SMD:C_0402_1005Metric"
 			(at 207.9752 113.03 0)
 			(effects
@@
 			)
 		)
-		(property "Footprint" "Resistor_SMD:R_0201_0603Metric"
+		(property "Footprint" "Resistor_SMD:R_0402_1005Metric"
 			(at 100.584 145.034 90)
 			(effects
@@
 			)
 		)
-		(property "Footprint" "Capacitor_SMD:C_0201_0603Metric"
+		(property "Footprint" "Capacitor_SMD:C_0402_1005Metric"
 			(at 239.7252 120.65 0)
 			(effects
@@
 			)
 		)
-		(property "Footprint" "Resistor_SMD:R_0201_0603Metric"
+		(property "Footprint" "Resistor_SMD:R_0402_1005Metric"
 			(at 151.384 152.654 90)
 			(effects
@@
 			)
 		)
-		(property "Footprint" "Resistor_SMD:R_0201_0603Metric"
+		(property "Footprint" "Resistor_SMD:R_0402_1005Metric"
 			(at 107.696 68.834 90)
 			(effects
@@
 			)
 		)
-		(property "Footprint" "Capacitor_SMD:C_0201_0603Metric"
+		(property "Footprint" "Capacitor_SMD:C_0402_1005Metric"
 			(at 168.6052 101.6 0)
 			(effects
@@
 			)
 		)
-		(property "Footprint" "Resistor_SMD:R_0201_0603Metric"
+		(property "Footprint" "Resistor_SMD:R_0402_1005Metric"
 			(at 140.716 169.164 90)
 			(effects
@@
 			)
 		)
-		(property "Footprint" "Resistor_SMD:R_0201_0603Metric"
+		(property "Footprint" "Resistor_SMD:R_0402_1005Metric"
 			(at 104.394 169.926 90)
 			(effects
@@
 			)
 		)
-		(property "Footprint" "Resistor_SMD:R_0201_0603Metric"
+		(property "Footprint" "Resistor_SMD:R_0402_1005Metric"
 			(at 147.574 53.086 90)
 			(effects
@@
 			)
 		)
-		(property "Footprint" "Resistor_SMD:R_0201_0603Metric"
+		(property "Footprint" "Resistor_SMD:R_0402_1005Metric"
 			(at 87.884 160.274 90)
 			(effects

Commit message: this is an electricity PCB
Connections:
- net GND: now also J3.2 (Pin_2); no longer J3.1 (Pin_1)
- net battery_in: now also J3.1 (Pin_1); no longer J3.2 (Pin_2)
Other:
- note added: "Charger/Power path selector"
- note added: "Fuel gauge"
- note added: "Voltage regulator"
- moved on the sheet: J3
Changed lines of the file:
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@@
 	(generator_version "9.0")
 	(paper "A4")
+	(text "Voltage regulator\n"
+		(exclude_from_sim no)
+		(at 199.898 90.424 0)
+		(effects
+			(font
+				(size 1.778 1.778)
+			)
+		)
+	)
+	(text "Charger/Power path selector"
+		(exclude_from_sim no)
+		(at 109.728 119.634 0)
+		(effects
+			(font
+				(size 1.778 1.778)
+			)
+		)
+	)
+	(text "Fuel gauge"
+		(exclude_from_sim no)
+		(at 126.746 22.098 0)
+		(effects
+			(font
+				(size 1.778 1.778)
+			)
+		)
+	)
 	(junction
 		(at 54.61 93.98)
@@
 	(wire
 		(pts
+			(xy 205.74 53.34) (xy 219.71 53.34)
+		)
+		(stroke
+			(width 0)
+			(type default)
+		)
+	)
+	(wire
+		(pts
 			(xy 104.14 54.61) (xy 110.49 54.61)
 		)
@@
 	(wire
 		(pts
-			(xy 214.63 53.34) (xy 218.44 53.34)
-		)
-		(stroke
-			(width 0)
-			(type default)
-		)
-	)
-	(wire
-		(pts
 			(xy 57.15 86.36) (xy 73.66 86.36)
 		)
@@
 	(wire
 		(pts
+			(xy 205.74 50.8) (xy 210.82 50.8)
+		)
+		(stroke
+			(width 0)
+			(type default)
+		)
+	)
+	(wire
+		(pts
 			(xy 200.66 105.41) (xy 207.01 105.41)
 		)
@@
 		(pts
 			(xy 105.41 133.35) (xy 105.41 140.97)
-		)
-		(stroke
-			(width 0)
-			(type default)
-		)
-	)
-	(wire
-		(pts
-			(xy 214.63 55.88) (xy 218.44 55.88)
 		)
 		(stroke
@@
 	)
 	(label "battery_in"
-		(at 218.44 53.34 0)
+		(at 219.71 53.34 0)
 		(effects
 			(font
@@
 	(symbol
 		(lib_id "Connector_Generic:Conn_01x02")
-		(at 209.55 55.88 180)
+		(at 200.66 53.34 180)
 		(unit 1)
 		(exclude_from_sim no)
@@
 		(fields_autoplaced yes)
 		(property "Reference" "J3"
-			(at 209.55 46.99 0)
+			(at 200.66 44.45 0)
 			(effects
 				(font
@@
 		)
 		(property "Value" "battery_con"
-			(at 209.55 49.53 0)
+			(at 200.66 46.99 0)
 			(effects
 				(font
@@
 		)
 		(property "Footprint" "Connector_JST:JST_PH_S2B-PH-K_1x02_P2.00mm_Horizontal"
-			(at 209.55 55.88 0)
+			(at 200.66 53.34 0)
 			(effects
 				(font
@@
 		)
 		(property "Datasheet" "~"
-			(at 209.55 55.88 0)
+			(at 200.66 53.34 0)
 			(effects
 				(font
@@
 		)
 		(property "Description" "Generic connector, single row, 01x02, script generated (kicad-library-utils/schlib/autogen/connector/)"
-			(at 209.55 55.88 0)
+			(at 200.66 53.34 0)
 			(effects
 				(font
@@
 	(symbol
 		(lib_id "power:GND")
-		(at 218.44 55.88 90)
+		(at 210.82 50.8 90)
 		(unit 1)
 		(exclude_from_sim no)
@@
 		(fields_autoplaced yes)
 		(property "Reference" "#PWR018"
-			(at 224.79 55.88 0)
+			(at 217.17 50.8 0)
 			(effects
 				(font
@@
 		)
 		(property "Value" "GND"
-			(at 222.25 55.8799 90)
+			(at 214.63 50.7999 90)
 			(effects
 				(font
@@
 		)
 		(property "Footprint" ""
-			(at 218.44 55.88 0)
+			(at 210.82 50.8 0)
 			(effects
 				(font
@@
 		)
 		(property "Datasheet" ""
-			(at 218.44 55.88 0)
+			(at 210.82 50.8 0)
 			(effects
 				(font
@@
 		)
 		(property "Description" "Power symbol creates a global label with name \"GND\" , ground"
-			(at 218.44 55.88 0)
-			(effects
-				(font
+			(at 210.82 50.8 0)
+			(effects
+				(font

Commit message: electroscity
Parts:
- removed R9: 10k, Resistor_SMD:R_0402_1005Metric, symbol Device:R_US
Changed lines of the file:
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@@
 	)
 	(junction
-		(at 139.7 161.29)
-		(diameter 0)
-		(color 0 0 0 0)
-	)
-	(junction
 		(at 104.14 39.37)
 		(diameter 0)
@@
 	(wire
 		(pts
-			(xy 139.7 172.72) (xy 139.7 175.26)
-		)
-		(stroke
-			(width 0)
-			(type default)
-		)
-	)
-	(wire
-		(pts
 			(xy 57.15 86.36) (xy 57.15 76.2)
 		)
@@
 	(wire
 		(pts
-			(xy 133.35 161.29) (xy 139.7 161.29)
+			(xy 133.35 161.29) (xy 147.32 161.29)
 		)
 		(stroke
@@
 	(wire
 		(pts
-			(xy 139.7 161.29) (xy 139.7 165.1)
-		)
-		(stroke
-			(width 0)
-			(type default)
-		)
-	)
-	(wire
-		(pts
-			(xy 139.7 161.29) (xy 147.32 161.29)
-		)
-		(stroke
-			(width 0)
-			(type default)
-		)
-	)
-	(wire
-		(pts
 			(xy 95.25 166.37) (xy 95.25 168.91)
 		)
@@
 		)
 	)
-	(label "+3.3V"
-		(at 139.7 175.26 270)
-		(effects
-			(font
-				(size 1.27 1.27)
-			)
-			(justify right bottom)
-		)
-	)
 	(hierarchical_label "ESP_SDA"
 		(shape output)
@@
 					(unit 1)
 				)
-			)
-		)
-	)
-	(symbol
-		(lib_id "Device:R_US")
-		(at 139.7 168.91 0)
-		(unit 1)
-		(exclude_from_sim no)
-		(in_bom yes)
-		(on_board yes)
-		(dnp no)
-		(fields_autoplaced yes)
-		(property "Reference" "R9"
-			(at 142.24 167.6399 0)
-			(effects
-				(font
-					(size 1.27 1.27)
-				)
-				(justify left)
-			)
-		)
-		(property "Value" "10k"
-			(at 142.24 170.1799 0)
-			(effects
-				(font
-					(size 1.27 1.27)
-				)
-				(justify left)
-			)
-		)
-		(property "Footprint" "Resistor_SMD:R_0402_1005Metric"
-			(at 140.716 169.164 90)
-			(effects
-				(font
-					(size 1.27 1.27)
-				)
-				(hide yes)
-			)
-		)
-		(property "Datasheet" "~"
-			(at 139.7 168.91 0)
-			(effects
-				(font
-					(size 1.27 1.27)
-				)
-				(hide yes)
-			)
-		)
-		(property "Description" "Resistor, US symbol"
-			(at 139.7 168.91 0)
-			(effects
-				(font
-					(size 1.27 1.27)
-				)
-				(hide yes)
-			)
-		)
-		(pin "1"
-		)
-		(pin "2"
-		)
-		(instances
-			(project "templog_mainboard"
-				(path "/84b25dc3-cc11-42e1-888d-24c6d5a62713/d593db04-482a-483f-ba64-3cc83809d23e"
-					(reference "R9")
-					(unit 1)
-				)
