File: templog_mainboard/power_mgmt.kicad_sch (KiCad schematic)
At the start: 29 parts, among them J1 USB_C_Receptacle_USB2.0_16P, J3 battery_con, U4 BQ27441-G1, U5 BQ24075RGT, U7 USBLC6-2SC6, U8 ADP2303ARDZ-3.3

Commit message: :ASEDfasef
Parts:
- removed C11, C12: 47uf, Capacitor_SMD:C_0402_1005Metric, symbol Device:C
- removed R11, R12: 31.6k, Resistor_SMD:R_0402_1005Metric, symbol Device:R_US
- removed R13: 100k, Resistor_SMD:R_0402_1005Metric, symbol Device:R_US
- removed SSB43L1: D, Diode_SMD:D_SMB, symbol Device:D
- removed U8: ADP2303ARDZ-3.3, Package_SO:SOIC-8-1EP_3.9x4.9mm_P1.27mm_EP2.29x3mm, symbol Regulator_Switching:ADP2303ARDZ-3.3
- added U8: TPS62203DBV, Package_TO_SOT_SMD:SOT-23-5, symbol Regulator_Switching:TPS62203DBV
- C10: value 0.1uf -> 10uf; footprint Capacitor_SMD:C_0402_1005Metric -> Capacitor_SMD:C_0805_2012Metric
- C9: footprint Capacitor_SMD:C_0402_1005Metric -> Capacitor_SMD:C_0805_2012Metric
- L1: value 4.7uH -> 10uH
Connections:
- net +3.3Vout: now also C10.2, U8.4 (FB)
- net GND: now also C10.1, U8.2 (GND)
- net powerpath_out: now also U8.1 (VI), U8.3 (EN)
- net at L1.1: now also U8.5 (SW); no longer C10.2

Commit message: electractiyt
Parts:
- C6: footprint Capacitor_SMD:C_0402_1005Metric -> Capacitor_SMD:C_0603_1608Metric
Connections:
- net +5VUSB: now also U7.5 (VBUS); no longer U7.2 (GND)
- net GND: now also U7.2 (GND); no longer U7.5 (VBUS)
- net USB_d+: now also U7.3 (I/O2); no longer U7.6 (I/O1)
Other:
- moved on the sheet: U7
Changed lines of the file:
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@@
 	)
 	(junction
-		(at 226.06 107.95)
+		(at 76.2 93.98)
 		(diameter 0)
 		(color 0 0 0 0)
 	)
 	(junction
-		(at 58.42 93.98)
+		(at 226.06 107.95)
 		(diameter 0)
 		(color 0 0 0 0)
@@
 	)
 	(junction
-		(at 57.15 99.06)
-		(diameter 0)
-		(color 0 0 0 0)
-	)
-	(junction
 		(at 38.1 119.38)
 		(diameter 0)
@@
 	)
 	(junction
+		(at 57.15 115.57)
+		(diameter 0)
+		(color 0 0 0 0)
+	)
+	(junction
 		(at 83.82 156.21)
 		(diameter 0)
@@
 	)
 	(no_connect
-		(at 72.39 106.68)
+		(at 72.39 110.49)
+	)
+	(no_connect
+		(at 62.23 110.49)
 	)
 	(no_connect
@@
 		(at 53.34 106.68)
 	)
-	(no_connect
-		(at 72.39 104.14)
-	)
 	(wire
 		(pts
@@
 	(wire
 		(pts
-			(xy 54.61 93.98) (xy 58.42 93.98)
-		)
-		(stroke
-			(width 0)
-			(type default)
-		)
-	)
-	(wire
-		(pts
 			(xy 205.74 53.34) (xy 219.71 53.34)
 		)
@@
 	(wire
 		(pts
-			(xy 60.96 104.14) (xy 62.23 104.14)
+			(xy 60.96 107.95) (xy 62.23 107.95)
 		)
 		(stroke
@@
 	(wire
 		(pts
-			(xy 58.42 93.98) (xy 58.42 106.68)
-		)
-		(stroke
-			(width 0)
-			(type default)
-		)
-	)
-	(wire
-		(pts
 			(xy 102.87 59.69) (xy 102.87 52.07)
 		)
@@
 	(wire
 		(pts
-			(xy 60.96 88.9) (xy 60.96 104.14)
+			(xy 60.96 88.9) (xy 60.96 107.95)
 		)
 		(stroke
@@
 	(wire
 		(pts
+			(xy 76.2 93.98) (xy 83.82 93.98)
+		)
+		(stroke
+			(width 0)
+			(type default)
+		)
+	)
+	(wire
+		(pts
 			(xy 101.6 59.69) (xy 102.87 59.69)
 		)
@@
 	(wire
 		(pts
-			(xy 105.41 140.97) (xy 107.95 140.97)
+			(xy 76.2 107.95) (xy 72.39 107.95)
 		)
 		(stroke
@@
 	(wire
 		(pts
-			(xy 96.52 40.64) (xy 107.95 40.64)
+			(xy 105.41 140.97) (xy 107.95 140.97)
 		)
 		(stroke
@@
 	(wire
 		(pts
-			(xy 209.55 107.95) (xy 214.63 107.95)
+			(xy 96.52 40.64) (xy 107.95 40.64)
 		)
 		(stroke
@@
 	(wire
 		(pts
-			(xy 133.35 161.29) (xy 147.32 161.29)
+			(xy 209.55 107.95) (xy 214.63 107.95)
 		)
 		(stroke
@@
 	(wire
 		(pts
-			(xy 57.15 76.2) (xy 53.34 76.2)
+			(xy 133.35 161.29) (xy 147.32 161.29)
 		)
 		(stroke
@@
 	(wire
 		(pts
-			(xy 123.19 64.77) (xy 123.19 66.04)
+			(xy 57.15 76.2) (xy 53.34 76.2)
 		)
 		(stroke
@@
 	(wire
 		(pts
-			(xy 53.34 93.98) (xy 54.61 93.98)
+			(xy 123.19 64.77) (xy 123.19 66.04)
 		)
 		(stroke
@@
 	(wire
 		(pts
-			(xy 106.68 72.39) (xy 106.68 76.2)
+			(xy 53.34 93.98) (xy 54.61 93.98)
 		)
 		(stroke
@@
 	(wire
 		(pts
-			(xy 58.42 106.68) (xy 62.23 106.68)
+			(xy 106.68 72.39) (xy 106.68 76.2)
 		)
 		(stroke
@@
 	(wire
 		(pts
-			(xy 57.15 99.06) (xy 67.31 99.06)
-		)
-		(stroke
-			(width 0)
-			(type default)
-		)
-	)
-	(wire
-		(pts
 			(xy 133.35 140.97) (xy 137.16 140.97)
 		)
@@
 	(wire
 		(pts
-			(xy 58.42 93.98) (xy 63.5 93.98)
+			(xy 54.61 93.98) (xy 76.2 93.98)
 		)
 		(stroke
@@
 	(wire
 		(pts
-			(xy 38.1 114.3) (xy 38.1 119.38)
+			(xy 76.2 93.98) (xy 76.2 107.95)
 		)
 		(stroke
@@
 	(wire
 		(pts
-			(xy 175.26 113.03) (xy 175.26 107.95)
+			(xy 38.1 114.3) (xy 38.1 119.38)
 		)
 		(stroke
@@
 	(wire
 		(pts
-			(xy 57.15 99.06) (xy 57.15 86.36)
+			(xy 175.26 113.03) (xy 175.26 107.95)
 		)
 		(stroke
@@
 	(wire
 		(pts
-			(xy 120.65 166.37) (xy 120.65 170.18)
+			(xy 57.15 86.36) (xy 57.15 115.57)
 		)
 		(stroke
@@
 	(wire
 		(pts
-			(xy 123.19 66.04) (xy 125.73 66.04)
+			(xy 120.65 166.37) (xy 120.65 170.18)
 		)
 		(stroke
@@
 	(wire
 		(pts
-			(xy 157.48 107.95) (xy 165.1 107.95)
+			(xy 123.19 66.04) (xy 125.73 66.04)
 		)
 		(stroke
@@
 	(wire
 		(pts
-			(xy 57.15 119.38) (xy 57.15 99.06)
+			(xy 157.48 107.95) (xy 165.1 107.95)
 		)
 		(stroke
@@
 	(wire
 		(pts
+			(xy 57.15 115.57) (xy 57.15 119.38)
+		)
+		(stroke
+			(width 0)
+			(type default)
+		)
+	)
+	(wire
+		(pts
 			(xy 105.41 161.29) (xy 105.41 166.37)
 		)
@@
 	(wire
 		(pts
-			(xy 67.31 111.76) (xy 67.31 114.3)
+			(xy 165.1 107.95) (xy 175.26 107.95)
 		)
 		(stroke
@@
 	(wire
 		(pts
-			(xy 165.1 107.95) (xy 175.26 107.95)
+			(xy 67.31 101.6) (xy 67.31 102.87)
 		)
 		(stroke
@@
 	(wire
 		(pts
+			(xy 57.15 115.57) (xy 67.31 115.57)
+		)
+		(stroke
+			(width 0)
+			(type default)
+		)
+	)
+	(wire
+		(pts
 			(xy 148.59 57.15) (xy 148.59 63.5)
 		)
@@
 	(hierarchical_label "USB_d+"
 		(shape output)
-		(at 63.5 93.98 0)
+		(at 83.82 93.98 0)
 		(effects
 			(font
@@
 			)
 		)
-		(property "Footprint" "Capacitor_SMD:C_0402_1005Metric"
+		(property "Footprint" "Capacitor_SMD:C_0603_1608Metric"
 			(at 43.18 120.3452 0)
 			(effects
@@
 	(symbol
 		(lib_id "Power_Protection:USBLC6-2SC6")
-		(at 67.31 106.68 180)
+		(at 67.31 110.49 180)
 		(unit 1)
 		(exclude_from_sim no)
@@
 		(fields_autoplaced yes)
 		(property "Reference" "U7"
-			(at 70.4281 96.52 0)
+			(at 70.4281 100.33 0)
 			(effects
 				(font
@@
 		)
 		(property "Value" "USBLC6-2SC6"
-			(at 70.4281 99.06 0)
+			(at 70.4281 102.87 0)
 			(effects
 				(font
@@
 		)
 		(property "Footprint" "Package_TO_SOT_SMD:SOT-23-6"
-			(at 66.04 100.33 0)
+			(at 66.04 104.14 0)
 			(effects
 				(font
@@
 		)
 		(property "Datasheet" "https://www.st.com/resource/en/datasheet/usblc6-2.pdf"
-			(at 66.04 98.425 0)
+			(at 66.04 102.235 0)
 			(effects
 				(font
@@
 		)
 		(property "Description" "Very low capacitance ESD protection diode, 2 data-line, SOT-23-6"
-			(at 67.31 106.68 0)
+			(at 67.31 110.49 0)
 			(effects
 				(font
@@
 	(symbol
 		(lib_id "power:GND")
-		(at 67.31 114.3 0)
+		(at 67.31 101.6 180)
 		(unit 1)
 		(exclude_from_sim no)
@@
 		(fields_autoplaced yes)
 		(property "Reference" "#PWR017"
-			(at 67.31 120.65 0)
+			(at 67.31 95.25 0)
 			(effects
 				(font
@@
 		)
 		(property "Value" "GND"
-			(at 67.31 119.38 0)
+			(at 67.31 96.52 0)
 			(effects
 				(font
@@
 		)
 		(property "Footprint" ""
-			(at 67.31 114.3 0)
+			(at 67.31 101.6 0)
 			(effects
 				(font
@@
 		)
 		(property "Datasheet" ""
-			(at 67.31 114.3 0)
+			(at 67.31 101.6 0)
 			(effects
 				(font
@@
 		)
 		(property "Description" "Power symbol creates a global label with name \"GND\" , ground"
-			(at 67.31 114.3 0)
+			(at 67.31 101.6 0)
 			(effects
 				(font
